Commit message: fix omnicar xacro ros2 control tag

File: urdf/omnicar_ignition.xacro (robot description, xacro)
@@ -6,10 +6,10 @@
             <material>Gazebo/White</material>
         </gazebo>
-        <ros2_control name="IgnitionSystem" type="system">
+        <ros2_control name="GazeboSystem" type="system">
             <hardware>
-                <plugin>ign_ros2_control/IgnitionSystem</plugin>
+                <plugin>gz_ros2_control/GazeboSimSystem</plugin>
             </hardware>
             <joint name="LH_WHEEL_JNT">
-                <command_interface name="effort" />
+                <command_interface name="velocity" />
                 <state_interface name="position">
                     <param name="initial_value">0.0</param>
@@ -21,5 +21,5 @@
             </joint>
             <joint name="LF_WHEEL_JNT">
-                <command_interface name="effort" />
+                <command_interface name="velocity" />
                 <state_interface name="position">
                     <param name="initial_value"> 0.0</param>
@@ -31,5 +31,5 @@
             </joint>
             <joint name="RH_WHEEL_JNT">
-                <command_interface name="effort" />
+                <command_interface name="velocity" />
                 <state_interface name="position">
                     <param name="initial_value">0.0</param>
@@ -41,5 +41,5 @@
             </joint>
             <joint name="RF_WHEEL_JNT">
-                <command_interface name="effort" />
+                <command_interface name="velocity" />
                 <state_interface name="position">
                     <param name="initial_value">0.0</param>
@@ -52,5 +52,5 @@
         </ros2_control>
         <gazebo>
-            <plugin filename="ign_ros2_control-system" name="ign_ros2_control::IgnitionROS2ControlPlugin">
+            <plugin filename="gz_ros2_control-system" name="gz_ros2_control::GazeboSimROS2ControlPlugin">
                 <parameters>$(find mulinex_ignition)/config/omnicar.yaml</parameters>
             </plugin>

File: urdf/wheel.xacro (robot description, xacro)
@@ -8,5 +8,5 @@
         <!-- Transformation based on the position of each link -->
     <xacro:macro name="wheel" params="prefix gazebo">
-        <joint name="${prefix}_WHEEL_" type="continuous">
+        <joint name="${prefix}_WHEEL_JNT" type="continuous">
                 <parent link="${prefix}_SHOULDER" />
                 <child link="${prefix}_WHEEL" />
