Commit message: update urdf to add robot namespace

File: urdf/imu_sensor.xacro (robot description, xacro)
@@ -13,5 +13,5 @@
     <xacro:property name="imu_len_z" value="0.01" />
     <xacro:include filename="$(find mulinex_description)/urdf/base_inertia.xacro" />
-    <xacro:macro name="imu_sensor" params="">
+    <xacro:macro name="imu_sensor" params="namespace">
         <joint name="base2imu" type="fixed">
             <parent link="base_link"/>
@@ -39,5 +39,5 @@
                     <update_rate>100</update_rate>
                     <visualize>true</visualize>
-                    <topic>imu</topic>
+                    <topic>${namespace}/imu</topic>
                     <plugin filename="libignition-gazebo-imu-system.so"
                             name="ignition::gazebo::systems::Imu">

File: urdf/lidar_sensor.xacro (robot description, xacro)
@@ -12,5 +12,5 @@
     <xacro:property name="lidar_len_h" value="0.055" />
     <xacro:include filename="$(find mulinex_description)/urdf/base_inertia.xacro" />
-    <xacro:macro name="lidar_sensor" params="tredi">
+    <xacro:macro name="lidar_sensor" params="tredi namespace">
         <joint name="base2lidar" type="fixed">
             <parent link="base_link"/>
@@ -43,5 +43,5 @@
                     <update_rate>10</update_rate>
                     <update_on_paused_sim>false</update_on_paused_sim>
-                    <topic>rgl_lidar</topic>
+                    <topic>${namespace}/rgl_lidar</topic>
                     <frame>lidar_link</frame>
                     <pattern_preset>Alpha Prime</pattern_preset>

File: urdf/omnicar.xacro (robot description, xacro)
@@ -11,4 +11,5 @@
     <xacro:arg name="yaml_file" default=""/>
     <xacro:arg name="lidar_3D" default="true"/>
+    <xacro:arg name="omnicar_namespace" default="omnicar"/>
     <xacro:arg name="jnt_prefix" default=""/>
     <xacro:arg name="front_haa" default="0.0" />
@@ -43,8 +44,8 @@
             <dimensions>3</dimensions>
             <odom_publish_frequency>100</odom_publish_frequency>
-            <odom_frame>gt_odom</odom_frame>
-            <robot_base_frame>base_link</robot_base_frame>
-            <odom_topic>gt_odom</odom_topic>
-            <tf_topic>gt_pose_gazebo</tf_topic>
+            <odom_frame>$(arg omnicar_namespace)/gt_odom</odom_frame>
+            <robot_base_frame>$(arg omnicar_namespace)/base_link</robot_base_frame>
+            <odom_topic>$(arg omnicar_namespace)/gt_odom</odom_topic>
+            <tf_topic>$(arg omnicar_namespace)/gt_pose_gazebo</tf_topic>
         </plugin>
         <!-- <plugin
@@ -85,7 +86,7 @@
         simplify_meshes="true"
     />
-    <xacro:imu_sensor/>
-    <xacro:lidar_sensor tredi="$(arg lidar_3D)"/>
-    <xacro:camera_sensor/>
+    <xacro:imu_sensor namespace="$(arg omnicar_namespace)"/>
+    <xacro:lidar_sensor tredi="$(arg lidar_3D)" namespace="$(arg omnicar_namespace)"/>
+    <!-- <xacro:camera_sensor namespace="$(arg omnicar_namespace)"/> -->
     <xacro:omnicar_ign_hw
         gazebo="$(arg use_gazebo)"
