Commit message: Add placeholder mulinex white (new version)

File: urdf/leg.xacro (robot description, xacro)
@@ -3,5 +3,5 @@
     <xacro:include filename="$(find mulinex_description)/urdf/links.xacro" />
     <xacro:property name="PI" value="3.141592" />
-    <xacro:macro name="leg" params="prefix gazebo jnt_pref simplify_meshes feet_type">
+    <xacro:macro name="leg" params="prefix gazebo jnt_pref simplify_meshes feet_type hfe_offset:=0 kfe_offset:=0">
         <!-- Module 1 -->
         <xacro:hip
@@ -17,4 +17,5 @@
             jnt_pref="${jnt_pref}"
             simplify_meshes="${simplify_meshes}"
+            hfe_offset="${hfe_offset}"
         />
         <!-- Lower leg link -->
@@ -25,4 +26,5 @@
             simplify_meshes="${simplify_meshes}"
             feet_type="$(arg feet_type)"
+            kfe_offset="${kfe_offset}"
         />
     </xacro:macro>

File: urdf/links.xacro (robot description, xacro)
@@ -267,9 +267,9 @@
     </xacro:macro>
     <!-- UPPER LEG -->
-    <xacro:macro name="upper_leg" params="prefix gazebo jnt_pref simplify_meshes">
+    <xacro:macro name="upper_leg" params="prefix gazebo jnt_pref simplify_meshes hfe_offset:=0">
         <!-- Transformation based on the position of each link -->
         <xacro:if value="${prefix == 'LF'}">
             <xacro:property name="hip_to_upper_leg_xyz" value="${HAA_2_HFE_x} ${HAA_2_HFE_y} 0" />
-            <xacro:property name="hip_to_upper_leg_rpy" value="0 0 0" />
+            <xacro:property name="hip_to_upper_leg_rpy" value="0 ${hfe_offset} 0" />
             <xacro:property name="axis" value="0 1 0" />
         </xacro:if>
@@ -277,5 +277,5 @@
             value="${prefix == 'LH'}">
             <xacro:property name="hip_to_upper_leg_xyz" value="${-HAA_2_HFE_x} ${HAA_2_HFE_y} 0" />
-            <xacro:property name="hip_to_upper_leg_rpy" value="0 0 0" />
+            <xacro:property name="hip_to_upper_leg_rpy" value="0 ${hfe_offset} 0" />
             <xacro:property name="axis" value="0 1 0" />
         </xacro:if>
@@ -283,5 +283,5 @@
             value="${prefix == 'RF'}">
             <xacro:property name="hip_to_upper_leg_xyz" value="${HAA_2_HFE_x} ${-HAA_2_HFE_y} 0" />
-            <xacro:property name="hip_to_upper_leg_rpy" value="0 0 0" />
+            <xacro:property name="hip_to_upper_leg_rpy" value="0 ${-hfe_offset} 0" />
             <xacro:property name="axis" value="0 -1 0" />
         </xacro:if>
@@ -289,5 +289,5 @@
             value="${prefix == 'RH'}">
             <xacro:property name="hip_to_upper_leg_xyz" value="${-HAA_2_HFE_x} ${-HAA_2_HFE_y} 0" />
-            <xacro:property name="hip_to_upper_leg_rpy" value="0 0 0" />
+            <xacro:property name="hip_to_upper_leg_rpy" value="0 ${-hfe_offset} 0" />
             <xacro:property name="axis" value="0 -1 0" />
         </xacro:if>
@@ -443,5 +443,5 @@
     </xacro:macro>
     <!-- LOWER LEG -->
-    <xacro:macro name="lower_leg" params="prefix gazebo jnt_pref simplify_meshes feet_type">
+    <xacro:macro name="lower_leg" params="prefix gazebo jnt_pref simplify_meshes feet_type kfe_offset:=0">
         <!-- NORMAL FEET CONFIGURATION -->
         <xacro:if value="${feet_type == 'normal'}">
@@ -450,4 +450,5 @@
                 <xacro:property name="upper_to_lower_leg_xyz"
                     value="${HFE_2_KFE_x} ${HFE_2_KFE_y} 0" />
+                <xacro:property name="upper_to_lower_leg_rpy" value="0 ${kfe_offset} 0" />
                 <xacro:property name="axis" value="0 1 0" />
             </xacro:if>
@@ -456,4 +457,5 @@
                 <xacro:property name="upper_to_lower_leg_xyz"
                     value="${-HFE_2_KFE_x} ${HFE_2_KFE_y} 0" />
+                <xacro:property name="upper_to_lower_leg_rpy" value="0 ${kfe_offset} 0" />
                 <xacro:property name="axis" value="0 1 0" />
             </xacro:if>
@@ -462,4 +464,5 @@
                 <xacro:property name="upper_to_lower_leg_xyz"
                     value="${HFE_2_KFE_x} ${-HFE_2_KFE_y} 0" />
+                <xacro:property name="upper_to_lower_leg_rpy" value="0 ${-kfe_offset} 0" />
                 <xacro:property name="axis" value="0 -1 0" />
             </xacro:if>
@@ -468,7 +471,7 @@
                 <xacro:property name="upper_to_lower_leg_xyz"
                     value="${-HFE_2_KFE_x} ${-HFE_2_KFE_y} 0" />
+                <xacro:property name="upper_to_lower_leg_rpy" value="0 ${-kfe_offset} 0" />
                 <xacro:property name="axis" value="0 -1 0" />
             </xacro:if>
-            <xacro:property name="upper_to_lower_leg_rpy" value="0 0 0" />
             <!-- Knee joint -->
             <joint name="${prefix}_KFE" type="revolute">
@@ -712,4 +715,5 @@
                 <xacro:property name="upper_to_lower_leg_xyz"
                     value="${HFE_2_KFE_x} ${HFE_2_KFE_y} 0" />
+                <xacro:property name="upper_to_lower_leg_rpy" value="0 ${kfe_offset} 0" />
                 <xacro:property name="axis" value="0 1 0" />
             </xacro:if>
@@ -718,4 +722,5 @@
                 <xacro:property name="upper_to_lower_leg_xyz"
                     value="${-HFE_2_KFE_x} ${HFE_2_KFE_y} 0" />
+                <xacro:property name="upper_to_lower_leg_rpy" value="0 ${kfe_offset} 0" />
                 <xacro:property name="axis" value="0 1 0" />
             </xacro:if>
@@ -724,4 +729,5 @@
                 <xacro:property name="upper_to_lower_leg_xyz"
                     value="${HFE_2_KFE_x} ${-HFE_2_KFE_y} 0" />
+                <xacro:property name="upper_to_lower_leg_rpy" value="0 ${-kfe_offset} 0" />
                 <xacro:property name="axis" value="0 -1 0" />
             </xacro:if>
@@ -730,7 +736,7 @@
                 <xacro:property name="upper_to_lower_leg_xyz"
                     value="${-HFE_2_KFE_x} ${-HFE_2_KFE_y} 0" />
+                <xacro:property name="upper_to_lower_leg_rpy" value="0 ${-kfe_offset} 0" />
                 <xacro:property name="axis" value="0 -1 0" />
             </xacro:if>
-            <xacro:property name="upper_to_lower_leg_rpy" value="0 0 0" />
             <!-- Knee joint -->
             <joint name="${prefix}_KFE" type="revolute">
@@ -3045,4 +3051,5 @@
                 <xacro:property name="upper_to_lower_leg_xyz"
                     value="${HFE_2_KFE_x} ${HFE_2_KFE_y} 0" />
+                <xacro:property name="upper_to_lower_leg_rpy" value="0 ${kfe_offset} 0" />
                 <xacro:property name="axis" value="0 1 0" />
             </xacro:if>
@@ -3051,4 +3058,5 @@
                 <xacro:property name="upper_to_lower_leg_xyz"
                     value="${-HFE_2_KFE_x} ${HFE_2_KFE_y} 0" />
+                <xacro:property name="upper_to_lower_leg_rpy" value="0 ${kfe_offset} 0" />
                 <xacro:property name="axis" value="0 1 0" />
             </xacro:if>
@@ -3057,4 +3065,5 @@
                 <xacro:property name="upper_to_lower_leg_xyz"
                     value="${HFE_2_KFE_x} ${-HFE_2_KFE_y} 0" />
+                <xacro:property name="upper_to_lower_leg_rpy" value="0 ${-kfe_offset} 0" />
                 <xacro:property name="axis" value="0 -1 0" />
             </xacro:if>
@@ -3063,7 +3072,7 @@
                 <xacro:property name="upper_to_lower_leg_xyz"
                     value="${-HFE_2_KFE_x} ${-HFE_2_KFE_y} 0" />
+                <xacro:property name="upper_to_lower_leg_rpy" value="0 ${-kfe_offset} 0" />
                 <xacro:property name="axis" value="0 -1 0" />
             </xacro:if>
-            <xacro:property name="upper_to_lower_leg_rpy" value="0 0 0" />
             <!-- Knee joint -->
             <joint name="${prefix}_KFE" type="revolute">
@@ -3480,4 +3489,5 @@
                 <xacro:property name="upper_to_lower_leg_xyz"
                     value="${HFE_2_KFE_x} ${HFE_2_KFE_y} 0" />
+                <xacro:property name="upper_to_lower_leg_rpy" value="0 ${kfe_offset} 0" />
                 <xacro:property name="axis" value="0 1 0" />
             </xacro:if>
@@ -3486,4 +3496,5 @@
                 <xacro:property name="upper_to_lower_leg_xyz"
                     value="${-HFE_2_KFE_x} ${HFE_2_KFE_y} 0" />
+                <xacro:property name="upper_to_lower_leg_rpy" value="0 ${kfe_offset} 0" />
                 <xacro:property name="axis" value="0 1 0" />
             </xacro:if>
@@ -3492,4 +3503,5 @@
                 <xacro:property name="upper_to_lower_leg_xyz"
                     value="${HFE_2_KFE_x} ${-HFE_2_KFE_y} 0" />
+                <xacro:property name="upper_to_lower_leg_rpy" value="0 ${-kfe_offset} 0" />
                 <xacro:property name="axis" value="0 -1 0" />
             </xacro:if>
@@ -3498,7 +3510,7 @@
                 <xacro:property name="upper_to_lower_leg_xyz"
                     value="${-HFE_2_KFE_x} ${-HFE_2_KFE_y} 0" />
+                <xacro:property name="upper_to_lower_leg_rpy" value="0 ${-kfe_offset} 0" />
                 <xacro:property name="axis" value="0 -1 0" />
             </xacro:if>
-            <xacro:property name="upper_to_lower_leg_rpy" value="0 0 0" />
             <!-- Knee joint -->
             <joint name="${prefix}_KFE" type="revolute">
