Commit message: Update mulinex_white starting config

File: urdf/mulinex_white.xacro (robot description, xacro)
@@ -12,6 +12,6 @@
     <xacro:arg name="feet_type" default="omni"/>
     <xacro:arg name="jnt_prefix" default="" />
-    <xacro:arg name="front_haa" default="0.0" />
-    <xacro:arg name="hind_haa" default="0.0" />
+    <xacro:property name="HFE" value="0.74" />
+    <xacro:property name="KFE" value="0.8" />
     <xacro:arg name="RH_HFE" default="0.0" />
     <xacro:arg name="RH_KFE" default="0.0" />
@@ -52,6 +52,6 @@
         simplify_meshes="$(arg simplify_meshes_lower_leg)"
         feet_type="$(arg feet_type)"
-        hfe_offset="${PI}"
-        kfe_offset="${PI}"
+        hfe_offset="${PI + HFE}"
+        kfe_offset="${PI - KFE}"
         />
     <xacro:leg
@@ -61,6 +61,6 @@
         simplify_meshes="$(arg simplify_meshes_lower_leg)"
         feet_type="$(arg feet_type)"
-        hfe_offset="${PI}"
-        kfe_offset="${PI}"
+        hfe_offset="${PI - HFE}"
+        kfe_offset="${PI + KFE}"
         />
     <xacro:leg
@@ -70,6 +70,6 @@
         simplify_meshes="$(arg simplify_meshes_lower_leg)"
         feet_type="$(arg feet_type)"
-        hfe_offset="${PI}"
-        kfe_offset="${PI}"
+        hfe_offset="${PI + HFE}"
+        kfe_offset="${PI - KFE}"
         />
     <xacro:leg
@@ -79,6 +79,6 @@
         simplify_meshes="$(arg simplify_meshes_lower_leg)"
         feet_type="$(arg feet_type)"
-        hfe_offset="${PI}"
-        kfe_offset="${PI}"
+        hfe_offset="${PI - HFE}"
+        kfe_offset="${PI + KFE}"
         />
     <xacro:if value="$(arg use_gazebo)">
