Commit message: add xacro args

File: urdf/links.xacro (robot description, xacro)
@@ -211,5 +211,5 @@
             <origin xyz="${hip_to_upper_leg_xyz}" rpy="${hip_to_upper_leg_rpy}" />
             <axis xyz="${axis}" />
-            <limit effort="2.7" lower="-${PI}" upper="${PI}" velocity="1000" />
+            <limit effort="5.0" lower="-${PI}" upper="${PI}" velocity="1000" />
             <!-- <dynamics damping="0.7" friction="100.0" /> -->
         </joint>
@@ -363,5 +363,5 @@
             <origin xyz="${upper_to_lower_leg_xyz}" rpy="${upper_to_lower_leg_rpy}" />
             <axis xyz="${axis}" />
-            <limit effort="2.7" lower="-${PI}" upper="${PI}" velocity="1000" />
+            <limit effort="5.0" lower="-${PI}" upper="${PI}" velocity="1000" />
             <!-- <dynamics damping="0.7" friction="100.0" /> -->
         </joint>

File: urdf/mulinex.xacro (robot description, xacro)
@@ -4,15 +4,19 @@
     <xacro:include filename="$(find mulinex_description)/urdf/leg.xacro" />
     <xacro:include filename="$(find mulinex_description)/urdf/material.xacro" />
-    <xacro:property name="use_gazebo" value="true" />
-    <xacro:property name="simplify_meshes_lower_leg" value="true"/>
-    <xacro:property name="add_wheels" value="false"/>
-    <xacro:property name="jnt_prefix" value="" />
-    <xacro:property name="hind_haa" value="0.0" />
-    <xacro:property name="hind_hfe" value="0.0" />
-    <xacro:property name="hind_kfe" value="0.0" />
-    <xacro:property name="front_haa" value="0.0" />
-    <xacro:property name="front_hfe" value="0.0" />
-    <xacro:property name="front_kfe" value="0.0" />
-    <link name="${jnt_prefix}base_link">
+    <xacro:arg name="use_gazebo" default="true" />
+    <xacro:arg name="simplify_meshes_lower_leg" default="true"/>
+    <xacro:arg name="add_wheels" default="false"/>
+    <xacro:arg name="jnt_prefix" default="" />
+    <xacro:arg name="hind_haa" default="0.0" />
+    <xacro:arg name="RH_HFE" default="0.0" />
+    <xacro:arg name="RH_KFE" default="0.0" />
+    <xacro:arg name="front_haa" default="0.0" />
+    <xacro:arg name="RF_HFE" default="0.0" />
+    <xacro:arg name="RF_KFE" default="0.0" />
+    <xacro:arg name="LH_HFE" default="0.0" />
+    <xacro:arg name="LH_KFE" default="0.0" />
+    <xacro:arg name="LF_HFE" default="0.0" />
+    <xacro:arg name="LF_KFE" default="0.0" />
+    <link name="$(arg jnt_prefix)base_link">
         <visual>
             <material name="white" />
@@ -39,27 +43,27 @@
     <xacro:leg
         prefix="LH"
-        gazebo="${use_gazebo}"
-        jnt_pref="${jnt_prefix}"
-        simplify_meshes="${simplify_meshes_lower_leg}"
-        wheels="${add_wheels}" />
+        gazebo="$(arg use_gazebo)"
+        jnt_pref="$(arg jnt_prefix)"
+        simplify_meshes="$(arg simplify_meshes_lower_leg)"
+        wheels="$(arg add_wheels)" />
     <xacro:leg
         prefix="LF"
-        gazebo="${use_gazebo}"
-        jnt_pref="${jnt_prefix}"
-        simplify_meshes="${simplify_meshes_lower_leg}"
-        wheels="${add_wheels}" />
+        gazebo="$(arg use_gazebo)"
+        jnt_pref="$(arg jnt_prefix)"
+        simplify_meshes="$(arg simplify_meshes_lower_leg)"
+        wheels="$(arg add_wheels)" />
     <xacro:leg
         prefix="RF"
-        gazebo="${use_gazebo}"
-        jnt_pref="${jnt_prefix}"
-        simplify_meshes="${simplify_meshes_lower_leg}"
-        wheels="${add_wheels}" />
+        gazebo="$(arg use_gazebo)"
+        jnt_pref="$(arg jnt_prefix)"
+        simplify_meshes="$(arg simplify_meshes_lower_leg)"
+        wheels="$(arg add_wheels)" />
     <xacro:leg
         prefix="RH"
-        gazebo="${use_gazebo}"
-        jnt_pref="${jnt_prefix}"
-        simplify_meshes="${simplify_meshes_lower_leg}"
-        wheels="${add_wheels}" />
-    <xacro:if value="${use_gazebo}">
+        gazebo="$(arg use_gazebo)"
+        jnt_pref="$(arg jnt_prefix)"
+        simplify_meshes="$(arg simplify_meshes_lower_leg)"
+        wheels="$(arg add_wheels)" />
+    <xacro:if value="$(arg use_gazebo)">
         <gazebo reference="base_link">
             <material>Gazebo/White</material>
@@ -77,5 +81,5 @@
                 <command_interface name="effort" />
                 <state_interface name="position">
-                    <param name="initial_value">-${hind_haa}</param>
+                    <param name="initial_value">$(arg hind_haa)</param>
                 </state_interface>
                 <state_interface name="velocity">
@@ -87,5 +91,5 @@
                 <command_interface name="effort" />
                 <state_interface name="position">
-                    <param name="initial_value">${hind_hfe}</param>
+                    <param name="initial_value">$(arg LH_HFE)</param>
                 </state_interface>
                 <state_interface name="velocity">
@@ -97,5 +101,5 @@
                 <command_interface name="effort" />
                 <state_interface name="position">
-                    <param name="initial_value">${hind_kfe}</param>
+                    <param name="initial_value">$(arg LH_KFE)</param>
                 </state_interface>
                 <state_interface name="velocity">
@@ -107,5 +111,5 @@
                 <command_interface name="effort" />
                 <state_interface name="position">
-                    <param name="initial_value">-${front_haa}</param>
+                    <param name="initial_value">$(arg front_haa)</param>
                 </state_interface>
                 <state_interface name="velocity">
@@ -117,5 +121,5 @@
                 <command_interface name="effort" />
                 <state_interface name="position">
-                    <param name="initial_value">${front_hfe}</param>
+                    <param name="initial_value">$(arg LF_HFE)</param>
                 </state_interface>
                 <state_interface name="velocity">
@@ -127,5 +131,5 @@
                 <command_interface name="effort" />
                 <state_interface name="position">
-                    <param name="initial_value">${front_kfe}</param>
+                    <param name="initial_value">$(arg LF_KFE)</param>
                 </state_interface>
                 <state_interface name="velocity">
@@ -137,5 +141,5 @@
                 <command_interface name="effort" />
                 <state_interface name="position">
-                    <param name="initial_value">${hind_haa}</param>
+                    <param name="initial_value">$(arg hind_haa)</param>
                 </state_interface>
                 <state_interface name="velocity">
@@ -147,5 +151,5 @@
                 <command_interface name="effort" />
                 <state_interface name="position">
-                    <param name="initial_value">${hind_hfe}</param>
+                    <param name="initial_value">$(arg RH_HFE)</param>
                 </state_interface>
                 <state_interface name="velocity">
@@ -157,5 +161,5 @@
                 <command_interface name="effort" />
                 <state_interface name="position">
-                    <param name="initial_value">${hind_kfe}</param>
+                    <param name="initial_value">$(arg RH_KFE)</param>
                 </state_interface>
                 <state_interface name="velocity">
@@ -167,5 +171,5 @@
                 <command_interface name="effort" />
                 <state_interface name="position">
-                    <param name="initial_value">${front_haa}</param>
+                    <param name="initial_value">$(arg front_haa)</param>
                 </state_interface>
                 <state_interface name="velocity">
@@ -177,5 +181,5 @@
                 <command_interface name="effort" />
                 <state_interface name="position">
-                    <param name="initial_value">${front_hfe}</param>
+                    <param name="initial_value">$(arg RF_HFE)</param>
                 </state_interface>
                 <state_interface name="velocity">
@@ -187,5 +191,5 @@
                 <command_interface name="effort" />
                 <state_interface name="position">
-                    <param name="initial_value">${front_kfe}</param>
+                    <param name="initial_value">$(arg RF_KFE)</param>
                 </state_interface>
                 <state_interface name="velocity">
@@ -251,5 +255,5 @@
         </gazebo>
     </xacro:if>
-    <xacro:unless value="${use_gazebo}">
+    <xacro:unless value="$(arg use_gazebo)">
         <!-- <ros2_control name="SOLO12_WB_Interface" type="system">
             <hardware>
