Commit message: Added mechanum version of omniwheels configuration

File: urdf/links.xacro (robot description, xacro)
@@ -80,4 +80,23 @@
     <xacro:property name="goat_lower_foot_RH"
         value="file://$(find mulinex_description)/meshes//goat_lower_foot_RH.STL" />
+    <!-- OMNI MESHES -->
+    <xacro:property name="omni_lower_leg_LF"
+        value="file://$(find mulinex_description)/meshes//omni_lower_leg_LF.STL" />
+    <xacro:property name="omni_lower_leg_LH"
+        value="file://$(find mulinex_description)/meshes//omni_lower_leg_LH.STL" />
+    <xacro:property name="omni_lower_leg_RF"
+        value="file://$(find mulinex_description)/meshes//omni_lower_leg_RF.STL" />
+    <xacro:property name="omni_lower_leg_RH"
+        value="file://$(find mulinex_description)/meshes//omni_lower_leg_RH.STL" />
+    <xacro:property name="mulinex_roller"
+        value="file://$(find mulinex_description)/meshes//roller_1.STL" />
+    <xacro:property name="mulinex_mec_wheel_LF"
+        value="file://$(find mulinex_description)/meshes//mecanum_wheel_lf.STL" />
+    <xacro:property name="mulinex_mec_wheel_RF"
+        value="file://$(find mulinex_description)/meshes//mecanum_wheel_rf.STL" />
+    <xacro:property name="mulinex_mec_wheel_LH"
+        value="file://$(find mulinex_description)/meshes//mecanum_wheel_lh.STL" />
+    <xacro:property name="mulinex_mec_wheel_RH"
+        value="file://$(find mulinex_description)/meshes//mecanum_wheel_rh.STL" />
     <!--  -->
     <!-- EACH MACRO CONSISTS OF THE LINK AND ITS PREVIOUS JOINT -->
@@ -730,10 +749,5 @@
                         <origin xyz="0 0 0" rpy="0 ${-PI/2} 0" />
                         <geometry>
-                            <xacro:if value="${simplify_meshes}">
-                                <mesh filename="${mulinex_lower_leg_left}" />
-                            </xacro:if>
-                            <xacro:unless value="${simplify_meshes}">
-                                <mesh filename="${old_mulinex_lower_leg_left}" />
-                            </xacro:unless>
+                            <mesh filename="${mulinex_lower_leg_left}" />
                         </geometry>
                     </xacro:if>
@@ -741,10 +755,5 @@
                         <origin xyz="0 0 0" rpy="0 ${PI/2} 0" />
                         <geometry>
-                            <xacro:if value="${simplify_meshes}">
-                                <mesh filename="${mulinex_lower_leg_left}" />
-                            </xacro:if>
-                            <xacro:unless value="${simplify_meshes}">
-                                <mesh filename="${old_mulinex_lower_leg_left}" />
-                            </xacro:unless>
+                            <mesh filename="${mulinex_lower_leg_left}" />
                         </geometry>
                     </xacro:if>
@@ -752,10 +761,5 @@
                         <origin xyz="0 0 0" rpy="0 ${-PI/2} 0" />
                         <geometry>
-                            <xacro:if value="${simplify_meshes}">
-                                <mesh filename="${mulinex_lower_leg_right}" />
-                            </xacro:if>
-                            <xacro:unless value="${simplify_meshes}">
-                                <mesh filename="${old_mulinex_lower_leg_right}" />
-                            </xacro:unless>
+                            <mesh filename="${mulinex_lower_leg_right}" />
                         </geometry>
                     </xacro:if>
@@ -763,10 +767,5 @@
                         <origin xyz="0 0 0" rpy="0 ${PI/2} 0" />
                         <geometry>
-                            <xacro:if value="${simplify_meshes}">
-                                <mesh filename="${mulinex_lower_leg_right}" />
-                            </xacro:if>
-                            <xacro:unless value="${simplify_meshes}">
-                                <mesh filename="${old_mulinex_lower_leg_right}" />
-                            </xacro:unless>
+                            <mesh filename="${mulinex_lower_leg_right}" />
                         </geometry>
                     </xacro:if>
@@ -790,5 +789,5 @@
                             <origin xyz="0 0 0" rpy="0 ${-PI/2} 0" />
                             <geometry>
-                                <mesh filename="${mulinex_lower_leg_right}" />
+                                <mesh filename="${msphereulinex_lower_leg_right}" />
                             </geometry>
                         </xacro:if>
@@ -829,36 +828,52 @@
                 </collision>
                 <inertial>
-                    <mass value="0.046942" />
+                    <mass value="0.30551" />
                     <xacro:if value="${prefix == 'LF'}">
                         <origin
-                            xyz="0.0660893 0.0198901 -1.552593e-05"
-                            rpy="0 0 0" />
-                        <inertia ixx="5.140780e-06" ixy="1.089102e-05"
-                            ixz="2.468115e-08" iyy="0.00021242"
-                            iyz="2.702972e-09" izz="0.00021154" />
+                            xyz="0.17801 0.030272 1.8448E-05"
+                            rpy="0 0 0" />
+                        <inertia
+                            ixx="6.1505E-05"
+                            ixy="-1.5369E-05"
+                            ixz="-4.7734E-08"
+                            iyy="0.00054256"
+                            iyz="-1.9337E-08"
+                            izz="0.00051876" />
                     </xacro:if>
                     <xacro:if value="${prefix == 'LH'}">
                         <origin
-                            xyz="-0.0660893 0.0198901 1.552593e-05"
-                            rpy="0 0 0" />
-                        <inertia ixx="5.140780e-06" ixy="-1.089102e-05"
-                            ixz="2.46811e-08" iyy="0.0002124295"
-                            iyz="-2.702972e-09" izz="0.0002115478" />
+                            xyz="-0.17801 0.030272 -1.8448E-05"
+                            rpy="0 0 0" />
+                        <inertia
+                            ixx="6.1505E-05"
+                            ixy="1.5369E-05"
+                            ixz="-4.7734E-08"
+                            iyy="0.00054256"
+                            iyz="1.9337E-08"
+                            izz="0.00051876" />
                     </xacro:if>
                     <xacro:if value="${prefix == 'RF'}">
                         <origin
-                            xyz="0.0660893 -0.0198901 -1.552593e-05"
-                            rpy="0 0 0" />
-                        <inertia ixx="5.140780e-06" ixy="1.089102e-05"
-                            ixz="-2.468115e-08" iyy="0.00021242"
-                            iyz="-2.702972e-09" izz="0.00021154" />
+                            xyz="0.17801 -0.030272 -1.8448E-05"
+                            rpy="0 0 0" />
+                        <inertia
+                            ixx="6.1505E-05"
+                            ixy="1.5369E-05"
+                            ixz="4.7734E-08"
+                            iyy="0.00054256"
+                            iyz="-1.9337E-08"
+                            izz="0.00051876" />
                     </xacro:if>
                     <xacro:if value="${prefix == 'RH'}">
                         <origin
-                            xyz="-0.0660893 -0.0198901 1.552593e-05"
-                            rpy="0 0 0" />
-                        <inertia ixx="5.140780e-06" ixy="-1.089102e-05"
-                            ixz="-2.46811e-08" iyy="0.0002124295"
-                            iyz="2.702972e-09" izz="0.0002115478" />
+                            xyz="-0.17801 -0.030272 1.8448E-05"
+                            rpy="0 0 0" />
+                        <inertia
+                            ixx="6.1505E-05"
+                            ixy="-1.5369E-05"
+                            ixz="4.7734E-08"
+                            iyy="0.00054256"
+                            iyz="1.9337E-08"
+                            izz="0.00051876" />
                     </xacro:if>
                 </inertial>
@@ -893,17 +908,17 @@
                 <child link="${prefix}_WHEEL" />
                 <xacro:if value="${prefix == 'LF'}">
-                    <origin xyz="${KFE_2_FOOT_x} ${KFE_2_FOOT_y} 0" rpy="0 0 0" />
+                    <origin xyz="${KFE_2_FOOT_x} 0.01145 0" rpy="0 0 0" />
                     <axis xyz="0 1 0" />
                 </xacro:if>
                 <xacro:if value="${prefix == 'LH'}">
-                    <origin xyz="${-KFE_2_FOOT_x} ${KFE_2_FOOT_y} 0" rpy="0 0 0" />
+                    <origin xyz="${-KFE_2_FOOT_x} 0.01145 0" rpy="0 0 0" />
                     <axis xyz="0 1 0" />
                 </xacro:if>
                 <xacro:if value="${prefix == 'RF'}">
-                    <origin xyz="${KFE_2_FOOT_x} ${-KFE_2_FOOT_y} 0" rpy="0 0 0" />
+                    <origin xyz="${KFE_2_FOOT_x} -0.01145 0" rpy="0 0 0" />
                     <axis xyz="0 1 0" />
                 </xacro:if>
                 <xacro:if value="${prefix == 'RH'}">
-                    <origin xyz="${-KFE_2_FOOT_x} ${-KFE_2_FOOT_y} 0" rpy="0 0 0" />
+                    <origin xyz="${-KFE_2_FOOT_x} -0.01145 0" rpy="0 0 0" />
                     <axis xyz="0 1 0" />
                 </xacro:if>
@@ -912,17 +927,60 @@
                 <visual>
                     <material name="white" />
-                    <origin xyz="0 0 0" rpy="${PI/2} 0 0" />
-                    <geometry>
-                        <cylinder length="0.10" radius="0.015" />
-                    </geometry>
+                    <xacro:if value="${prefix == 'LF'}">
+                        <origin xyz="0 0 0" rpy="0 0 0" />
+                        <geometry>
+                            <mesh filename="${mulinex_mec_wheel_LF}" />
+                        </geometry>
+                    </xacro:if>
+                    <xacro:if value="${prefix == 'LH'}">
+                        <origin xyz="0 0  0" rpy="0 0 0" />
+                        <geometry>
+                            <mesh filename="${mulinex_mec_wheel_LH}" />
+                        </geometry>
+                    </xacro:if>
+                    <xacro:if value="${prefix == 'RF'}">
+                        <origin xyz="0 0 0" rpy="0 0 0" />
+                        <geometry>
+                            <mesh filename="${mulinex_mec_wheel_RF}" />
+                        </geometry>
+                    </xacro:if>
+                    <xacro:if value="${prefix == 'RH'}">
+                        <origin xyz="0 0 0" rpy="0 0 0" />
+                        <geometry>
+                            <mesh filename="${mulinex_mec_wheel_RH}" />
+                        </geometry>
+                    </xacro:if>
                 </visual>
-                <xacro:if value="${simplify_meshes}">
-                    <collision>
-                        <origin xyz="0 0 0" rpy="${PI/2} 0 0" />
-                        <geometry>
-                            <cylinder length="0.10" radius="0.015" />
-                        </geometry>
-                    </collision>
-                </xacro:if>
+                <!-- NO COLLISION FOR THE MECHANUM WHEELS -->
+                <inertial>
+                    <xacro:if value="${prefix == 'LF'}">
+                        <origin xyz="0 0.047255 -2.335E-07" rpy="0 0 0" />
+                        <mass value="0.078919" />
+                        <inertia ixx="4.9627E-05" ixy="1.7873E-11"
+                            ixz="-2.2576E-09" iyy="7.8948E-05"
+                            iyz="-7.6317E-12" izz="4.9622E-05" />
+                    </xacro:if>
+                    <xacro:if value="${prefix == 'LH'}">
+                        <origin xyz="0 0.047255 -1.5525E-07" rpy="0 0 0" />
+                        <mass value="0.078525" />
+                        <inertia ixx="4.9627E-05" ixy="-2.1009E-12"
+                            ixz="-1.8882E-09" iyy="7.8948E-05"
+                            iyz="4.4431E-12" izz="4.9622E-05" />
+                    </xacro:if>
+                    <xacro:if value="${prefix == 'RF'}">
+                        <origin xyz="0 -0.047255 -1.5525E-07" rpy="0 0 0" />
+                        <mass value="0.078525" />
+                        <inertia ixx="4.9627E-05" ixy="-2.1009E-12"
+                            ixz="1.8882E-09" iyy="7.8948E-05"
+                            iyz="-4.4431E-12" izz="4.9622E-05" />
+                    </xacro:if>
+                    <xacro:if value="${prefix == 'RH'}">
+                        <origin xyz="0 -0.047255 -2.3351E-07" rpy="0 0 0" />
+                        <mass value="0.078919" />
+                        <inertia ixx="4.9627E-05" ixy="1.7873E-11"
+                            ixz="-2.2576E-09" iyy="7.8948E-05"
+                            iyz="-7.6317E-12" izz="4.9622E-05" />
+                    </xacro:if>
+                </inertial>
             </link>
             <xacro:if value="${gazebo}">
@@ -948,4 +1006,178 @@
                         </surface>
                     </collision>
+                </gazebo>
+            </xacro:if>
+            <link name="${prefix}_Roller1">
+                <xacro:if value="${prefix == 'LF'}">
+                    <inertial>
+                        <origin
+                            xyz="0 0 6.3075E-15"
+                            rpy="0 0 0" />
+                        <mass
+                            value="0.0059616" />
+                        <inertia
+                            ixx="7.911E-07"
+                            ixy="1.2914E-12"
+                            ixz="1.2242E-22"
+                            iyy="7.9113E-07"
+                            iyz="-5.294E-23"
+                            izz="2.3532E-07" />
+                    </inertial>
+                    <visual>
+                        <origin
+                            xyz="0 0 0"
+                            rpy="0 0 0" />
+                        <geometry>
+                            <mesh filename="${mulinex_roller}" />
+                        </geometry>
+                        <material
+                            name="">
+                            <color
+                                rgba="0.29804 0.29804 0.29804 1" />
+                        </material>
+                    </visual>
+                    <collision>
+                        <origin
+                            xyz="0 0 0"
+                            rpy="0 0 0" />
+                        <geometry>
+                            <mesh filename="${mulinex_roller}" />
+                        </geometry>
+                    </collision>
+                </xacro:if>
+                <xacro:if value="${prefix == 'RF'}">
+                    <inertial>
+                        <origin
+                            xyz="0 0 0"
+                            rpy="0 0 0" />
+                        <mass
+                            value="0.0059616" />
+                        <inertia
+                            ixx="7.911E-07"
+                            ixy="1.2914E-12"
+                            ixz="2.5808E-22"
+                            iyy="7.9113E-07"
+                            iyz="-5.4263E-22"
+                            izz="2.3532E-07" />
+                    </inertial>
+                    <visual>
+                        <origin
+                            xyz="0 0 0"
+                            rpy="0 0 0" />
+                        <geometry>
+                            <mesh filename="${mulinex_roller}" />
+                        </geometry>
+                        <material
+                            name="">
+                            <color
+                                rgba="0.29804 0.29804 0.29804 1" />
+                        </material>
+                    </visual>
+                    <collision>
+                        <origin
+                            xyz="0 0 0"
+                            rpy="0 0 0" />
+                        <geometry>
+                            <mesh filename="${mulinex_roller}" />
+                        </geometry>
+                    </collision>
+                </xacro:if>
+                <xacro:if value="${prefix == 'LH'}">
+                    <inertial>
+                        <origin
+                            xyz="0 0 6.3075E-15"
+                            rpy="0 0 0" />
+                        <mass
+                            value="0.0059616" />
+                        <inertia
+                            ixx="7.911E-07"
+                            ixy="1.2914E-12"
+                            ixz="1.9521E-22"
+                            iyy="7.9113E-07"
+                            iyz="-5.0954E-22"
+                            izz="2.3532E-07" />
+                    </inertial>
+                    <visual>
+                        <origin
+                            xyz="0 0 0"
+                            rpy="0 0 0" />
+                        <geometry>
+                            <mesh filename="${mulinex_roller}" />
+                        </geometry>
+                        <material
+                            name="">
+                            <color
+                                rgba="0.29804 0.29804 0.29804 1" />
+                        </material>
+                    </visual>
+                    <collision>
+                        <origin
+                            xyz="0 0 0"
+                            rpy="0 0 0" />
+                        <geometry>
+                            <mesh filename="${mulinex_roller}" />
+                        </geometry>
+                    </collision>
+                </xacro:if>
+                <xacro:if value="${prefix == 'RH'}">
+                    <inertial>
+                        <origin
+                            xyz="0 0 6.3075E-15"
+                            rpy="0 0 0" />
+                        <mass
+                            value="0.0059616" />
+                        <inertia
+                            ixx="7.911E-07"
+                            ixy="1.2914E-12"
+                            ixz="1.2242E-22"
+                            iyy="7.9113E-07"
+                            iyz="-5.294E-23"
+                            izz="2.3532E-07" />
+                    </inertial>
+                    <visual>
+                        <origin
+                            xyz="0 0 0"
+                            rpy="0 0 0" />
+                        <geometry>
+                            <mesh filename="${mulinex_roller}" />
+                        </geometry>
+                        <material
+                            name="">
+                            <color
+                                rgba="0.29804 0.29804 0.29804 1" />
+                        </material>
+                    </visual>
+                    <collision>
+                        <origin
+                            xyz="0 0 0"
+                            rpy="0 0 0" />
+                        <geometry>
+                            <mesh filename="${mulinex_roller}" />
+                        </geometry>
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
File: urdf/mulinex.xacro (robot description, xacro)
@@ -5,10 +5,10 @@
     <xacro:include filename="$(find mulinex_description)/urdf/material.xacro" />
     <xacro:arg name="use_gazebo" default="true" />
-    <xacro:arg name="simplify_meshes_lower_leg" default="false"/>
+    <xacro:arg name="simplify_meshes_lower_leg" default="true"/>
     <!-- use "normal" if normal feet are used
         use "omni" if omniwheels are used
         use "goat" if goat feet are used
         use "track" if track feet are used -->
-    <xacro:arg name="feet_type" default="goat"/>
+    <xacro:arg name="feet_type" default="omni"/>
     <xacro:arg name="jnt_prefix" default="" />
     <xacro:arg name="front_haa" default="0.0" />
