Commit message: update omnicar urdf and add ingition stuff

File: urdf/links.xacro (robot description, xacro)
@@ -695,5 +695,5 @@
                         </surface>
                     </collision>
-                    <sensor name="${prefix}_contactsensor_sensor" type="contact">
+                    <!-- <sensor name="${prefix}_contactsensor_sensor" type="contact">
                         <always_on>true</always_on>
                         <update_rate>50</update_rate>
@@ -702,5 +702,5 @@
                                 ${prefix}_LOWER_LEG_fixed_joint_lump__${prefix}_FOOT_collision_1</collision>
                         </contact>
-                    </sensor>
+                    </sensor> -->
                 </gazebo>
             </xacro:if>
@@ -1180,5 +1180,5 @@
                         </surface>
                     </collision>
-                    <sensor name="${prefix}_contactsensor_sensor" type="contact">
+                    <!-- <sensor name="${prefix}_contactsensor_sensor" type="contact">
                         <always_on>true</always_on>
                         <update_rate>50</update_rate>
@@ -1187,5 +1187,5 @@
                                 ${prefix}_LOWER_LEG_fixed_joint_lump__${prefix}_FOOT_collision_1</collision>
                         </contact>
-                    </sensor>
+                    </sensor> -->
                 </gazebo>
             </xacro:if>
@@ -1362,5 +1362,5 @@
                         </surface>
                     </collision>
-                    <sensor name="${prefix}_contactsensor_sensor" type="contact">
+                    <!-- <sensor name="${prefix}_contactsensor_sensor" type="contact">
                         <always_on>true</always_on>
                         <update_rate>50</update_rate>
@@ -1369,5 +1369,5 @@
                                 ${prefix}_LOWER_LEG_fixed_joint_lump__${prefix}_FOOT_collision_1</collision>
                         </contact>
-                    </sensor>
+                    </sensor> -->
                 </gazebo>
             </xacro:if>
@@ -1544,5 +1544,5 @@
                         </surface>
                     </collision>
-                    <sensor name="${prefix}_contactsensor_sensor" type="contact">
+                    <!-- <sensor name="${prefix}_contactsensor_sensor" type="contact">
                         <always_on>true</always_on>
                         <update_rate>50</update_rate>
@@ -1551,5 +1551,5 @@
                                 ${prefix}_LOWER_LEG_fixed_joint_lump__${prefix}_FOOT_collision_1</collision>
                         </contact>
-                    </sensor>
+                    </sensor> -->
                 </gazebo>
             </xacro:if>
@@ -1726,5 +1726,5 @@
                         </surface>
                     </collision>
-                    <sensor name="${prefix}_contactsensor_sensor" type="contact">
+                    <!-- <sensor name="${prefix}_contactsensor_sensor" type="contact">
                         <always_on>true</always_on>
                         <update_rate>50</update_rate>
@@ -1733,5 +1733,5 @@
                                 ${prefix}_LOWER_LEG_fixed_joint_lump__${prefix}_FOOT_collision_1</collision>
                         </contact>
-                    </sensor>
+                    </sensor> -->
                 </gazebo>
             </xacro:if>
@@ -1908,5 +1908,5 @@
                         </surface>
                     </collision>
-                    <sensor name="${prefix}_contactsensor_sensor" type="contact">
+                    <!-- <sensor name="${prefix}_contactsensor_sensor" type="contact">
                         <always_on>true</always_on>
                         <update_rate>50</update_rate>
@@ -1915,5 +1915,5 @@
                                 ${prefix}_LOWER_LEG_fixed_joint_lump__${prefix}_FOOT_collision_1</collision>
                         </contact>
-                    </sensor>
+                    </sensor> -->
                 </gazebo>
             </xacro:if>
@@ -2090,5 +2090,5 @@
                         </surface>
                     </collision>
-                    <sensor name="${prefix}_contactsensor_sensor" type="contact">
+                    <!-- <sensor name="${prefix}_contactsensor_sensor" type="contact">
                         <always_on>true</always_on>
                         <update_rate>50</update_rate>
@@ -2097,5 +2097,5 @@
                                 ${prefix}_LOWER_LEG_fixed_joint_lump__${prefix}_FOOT_collision_1</collision>
                         </contact>
-                    </sensor>
+                    </sensor> -->
                 </gazebo>
             </xacro:if>
@@ -2272,5 +2272,5 @@
                         </surface>
                     </collision>
-                    <sensor name="${prefix}_contactsensor_sensor" type="contact">
+                    <!-- <sensor name="${prefix}_contactsensor_sensor" type="contact">
                         <always_on>true</always_on>
                         <update_rate>50</update_rate>
@@ -2279,5 +2279,5 @@
                                 ${prefix}_LOWER_LEG_fixed_joint_lump__${prefix}_FOOT_collision_1</collision>
                         </contact>
-                    </sensor>
+                    </sensor> -->
                 </gazebo>
             </xacro:if>
@@ -2454,5 +2454,5 @@
                         </surface>
                     </collision>
-                    <sensor name="${prefix}_contactsensor_sensor" type="contact">
+                    <!-- <sensor name="${prefix}_contactsensor_sensor" type="contact">
                         <always_on>true</always_on>
                         <update_rate>50</update_rate>
@@ -2461,5 +2461,5 @@
                                 ${prefix}_LOWER_LEG_fixed_joint_lump__${prefix}_FOOT_collision_1</collision>
                         </contact>
-                    </sensor>
+                    </sensor> -->
                 </gazebo>
             </xacro:if>
@@ -2636,5 +2636,5 @@
                         </surface>
                     </collision>
-                    <sensor name="${prefix}_contactsensor_sensor" type="contact">
+                    <!-- <sensor name="${prefix}_contactsensor_sensor" type="contact">
                         <always_on>true</always_on>
                         <update_rate>50</update_rate>
@@ -2643,5 +2643,5 @@
                                 ${prefix}_LOWER_LEG_fixed_joint_lump__${prefix}_FOOT_collision_1</collision>
                         </contact>
-                    </sensor>
+                    </sensor> -->
                 </gazebo>
             </xacro:if>
@@ -2818,5 +2818,5 @@
                         </surface>
                     </collision>
-                    <sensor name="${prefix}_contactsensor_sensor" type="contact">
+                    <!-- <sensor name="${prefix}_contactsensor_sensor" type="contact">
                         <always_on>true</always_on>
                         <update_rate>50</update_rate>
@@ -2825,5 +2825,5 @@
                                 ${prefix}_LOWER_LEG_fixed_joint_lump__${prefix}_FOOT_collision_1</collision>
                         </contact>
-                    </sensor>
+                    </sensor> -->
                 </gazebo>
             </xacro:if>
@@ -3809,5 +3809,5 @@
                         </surface>
                     </collision>
-                    <sensor name="${prefix}_contactsensor_sensor" type="contact">
+                    <!-- <sensor name="${prefix}_contactsensor_sensor" type="contact">
                         <always_on>true</always_on>
                         <update_rate>50</update_rate>
@@ -3816,5 +3816,5 @@
                                 ${prefix}_LOWER_LEG_fixed_joint_lump__${prefix}_FOOT_collision_1</collision>
                         </contact>
-                    </sensor>
+                    </sensor> -->
                 </gazebo>
             </xacro:if>

File: urdf/omnicar.xacro (robot description, xacro)
@@ -2,6 +2,9 @@
 <robot name="mulinex" xmlns:xacro="http://ros.org/wiki/xacro">
     <xacro:include filename="$(find mulinex_description)/urdf/omni_car_module.xacro" />
-    <xacro:include filename="$(find mulinex_description)/urdf/material.xacro" />
-    <xacro:arg name="use_gazebo" default="false" />
+    <!-- <xacro:include filename="$(find mulinex_description)/urdf/material.xacro" /> -->
+    <xacro:include filename="$(find mulinex_description)/urdf/omnicar_gazebo.xacro" />
+    <xacro:include filename="$(find mulinex_description)/urdf/omnicar_ignition.xacro" />
+    <xacro:arg name="use_gazebo" default="true" />
+    <xacro:arg name="use_ignition" default="true" />
     <xacro:arg name="simplify_meshes_lower_leg" default="true"/>
     <xacro:arg name="jnt_prefix" default=""/>
@@ -68,112 +71,11 @@
     />
     <xacro:if value="$(arg use_gazebo)">
-        <gazebo reference="base_link">
-            <material>Gazebo/White</material>
-        </gazebo>
-        <gazebo>
-            <plugin filename="libgazebo_ros2_control.so" name="gazebo_ros2_control">
-                <parameters>$(find mulinex_gazebo)/config/mulinex_gazebo_sim_jnt_PD_IMU.yaml</parameters>
-            </plugin>
-        </gazebo>
-        <ros2_control name="GazeboSystem" type="system">
-            <hardware>
-                <plugin>gazebo_ros2_control/GazeboSystem</plugin>
-            </hardware>
-            <joint name="LH_WHEEL">
-                <command_interface name="effort" />
-                <state_interface name="position">
-                    <param name="initial_value">$(arg hind_haa)</param>
-                </state_interface>
-                <state_interface name="velocity">
-                    <param name="initial_value">0.0</param>
-                </state_interface>
-                <state_interface name="effort" />
-            </joint>
-            <joint name="LF_WHEEL">
-                <command_interface name="effort" />
-                <state_interface name="position">
-                    <param name="initial_value">$(arg front_haa)</param>
-                </state_interface>
-                <state_interface name="velocity">
-                    <param name="initial_value">0.0</param>
-                </state_interface>
-                <state_interface name="effort" />
-            </joint>
-            <joint name="RH_WHEEL">
-                <command_interface name="effort" />
-                <state_interface name="position">
-                    <param name="initial_value">$(arg hind_haa)</param>
-                </state_interface>
-                <state_interface name="velocity">
-                    <param name="initial_value">0.0</param>
-                </state_interface>
-                <state_interface name="effort" />
-            </joint>
-            <joint name="RF_WHEEL">
-                <command_interface name="effort" />
-                <state_interface name="position">
-                    <param name="initial_value">$(arg front_haa)</param>
-                </state_interface>
-                <state_interface name="velocity">
-                    <param name="initial_value">0.0</param>
-                </state_interface>
-                <state_interface name="effort" />
-            </joint>
-        </ros2_control>
-        <gazebo reference="base_link">
-            <sensor name="br_imu" type="imu">
-                <always_on>true</always_on>
-                <update_rate>100</update_rate>
-                <imu>
-                <angular_velocity>
-                    <x>
-                    <noise type="gaussian">
-                        <mean>0.0</mean>
-                        <stddev>2e-4</stddev>
-                    </noise>
-                    </x>
-                    <y>
-                    <noise type="gaussian">
-                        <mean>0.0</mean>
-                        <stddev>2e-4</stddev>
-                    </noise>
-                    </y>
-                    <z>
-                    <noise type="gaussian">
-                        <mean>0.0</mean>
-                        <stddev>2e-4</stddev>
-                    </noise>
-                    </z>
-                </angular_velocity>
-                <linear_acceleration>
-                    <x>
-                    <noise type="gaussian">
-                        <mean>0.0</mean>
-                        <stddev>1.7e-2</stddev>
-                    </noise>
-                    </x>
-                    <y>
-                    <noise type="gaussian">
-                        <mean>0.0</mean>
-                        <stddev>1.7e-2</stddev>
-                    </noise>
-                    </y>
-                    <z>
-                    <noise type="gaussian">
-                        <mean>0.0</mean>
-                        <stddev>1.7e-2</stddev>
-                    </noise>
-                    </z>
-                </linear_acceleration>
-                </imu>
-                <!-- <plugin name="bytes_imu" filename="libgazebo_ros_imu_sensor.so">
-                    <ros>
-                        <namespace>imu</namespace>
-                        <remapping>~/out:=data</remapping>
-                    </ros>
-                    <initial_orientation_as_reference>false</initial_orientation_as_reference>
-                </plugin> -->
-            </sensor>
-        </gazebo>
+        <xacro:if value="$(arg use_ignition)">
+            <xacro:omnicar_ign_hw
+                gazebo="$(arg use_ignition)"
+            />
+        </xacro:if>
+        <xacro:unless value="$(arg use_ignition)">
+        </xacro:unless>
     </xacro:if>
 </robot>

File: urdf/wheel.xacro (robot description, xacro)
@@ -8,5 +8,5 @@
         <!-- Transformation based on the position of each link -->
     <xacro:macro name="wheel" params="prefix gazebo">
-        <joint name="${prefix}_ANKLE" type="continuous">
+        <joint name="${prefix}_WHEEL_" type="continuous">
                 <parent link="${prefix}_SHOULDER" />
                 <child link="${prefix}_WHEEL" />
@@ -284,5 +284,5 @@
                         </surface>
                     </collision>
-                    <sensor name="${prefix}_contactsensor_sensor" type="contact">
+                    <!-- <sensor name="${prefix}_contactsensor_sensor" type="contact">
                         <always_on>true</always_on>
                         <update_rate>50</update_rate>
@@ -291,5 +291,5 @@
                                 ${prefix}_LOWER_LEG_fixed_joint_lump__${prefix}_FOOT_collision_1</collision>
                         </contact>
-                    </sensor>
+                    </sensor> -->
                 </gazebo>
             </xacro:if>
@@ -466,5 +466,5 @@
                         </surface>
                     </collision>
-                    <sensor name="${prefix}_contactsensor_sensor" type="contact">
+                    <!-- <sensor name="${prefix}_contactsensor_sensor" type="contact">
                         <always_on>true</always_on>
                         <update_rate>50</update_rate>
@@ -473,5 +473,5 @@
                                 ${prefix}_LOWER_LEG_fixed_joint_lump__${prefix}_FOOT_collision_1</collision>
                         </contact>
-                    </sensor>
+                    </sensor> -->
                 </gazebo>
             </xacro:if>
@@ -648,5 +648,5 @@
                         </surface>
                     </collision>
-                    <sensor name="${prefix}_contactsensor_sensor" type="contact">
+                    <!-- <sensor name="${prefix}_contactsensor_sensor" type="contact">
                         <always_on>true</always_on>
                         <update_rate>50</update_rate>
@@ -655,5 +655,5 @@
                                 ${prefix}_LOWER_LEG_fixed_joint_lump__${prefix}_FOOT_collision_1</collision>
                         </contact>
-                    </sensor>
+                    </sensor> -->
                 </gazebo>
             </xacro:if>
@@ -830,5 +830,5 @@
                         </surface>
                     </collision>
-                    <sensor name="${prefix}_contactsensor_sensor" type="contact">
+                    <!-- <sensor name="${prefix}_contactsensor_sensor" type="contact">
                         <always_on>true</always_on>
                         <update_rate>50</update_rate>
@@ -837,5 +837,5 @@
                                 ${prefix}_LOWER_LEG_fixed_joint_lump__${prefix}_FOOT_collision_1</collision>
                         </contact>
-                    </sensor>
+                    </sensor> -->
                 </gazebo>
             </xacro:if>
@@ -1012,5 +1012,5 @@
                         </surface>
                     </collision>
-                    <sensor name="${prefix}_contactsensor_sensor" type="contact">
+                    <!-- <sensor name="${prefix}_contactsensor_sensor" type="contact">
                         <always_on>true</always_on>
                         <update_rate>50</update_rate>
@@ -1019,5 +1019,5 @@
                                 ${prefix}_LOWER_LEG_fixed_joint_lump__${prefix}_FOOT_collision_1</collision>
                         </contact>
-                    </sensor>
+                    </sensor> -->
                 </gazebo>
             </xacro:if>
@@ -1194,5 +1194,5 @@
                         </surface>
                     </collision>
-                    <sensor name="${prefix}_contactsensor_sensor" type="contact">
+                    <!-- <sensor name="${prefix}_contactsensor_sensor" type="contact">
                         <always_on>true</always_on>
                         <update_rate>50</update_rate>
@@ -1201,5 +1201,5 @@
                                 ${prefix}_LOWER_LEG_fixed_joint_lump__${prefix}_FOOT_collision_1</collision>
                         </contact>
-                    </sensor>
+                    </sensor> -->
                 </gazebo>
             </xacro:if>
@@ -1376,5 +1376,5 @@
                         </surface>
                     </collision>
-                    <sensor name="${prefix}_contactsensor_sensor" type="contact">
+                    <!-- <sensor name="${prefix}_contactsensor_sensor" type="contact">
                         <always_on>true</always_on>
                         <update_rate>50</update_rate>
@@ -1383,5 +1383,5 @@
                                 ${prefix}_LOWER_LEG_fixed_joint_lump__${prefix}_FOOT_collision_1</collision>
                         </contact>
-                    </sensor>
+                    </sensor> -->
                 </gazebo>
             </xacro:if>
@@ -1558,5 +1558,5 @@
                         </surface>
                     </collision>
-                    <sensor name="${prefix}_contactsensor_sensor" type="contact">
+                    <!-- <sensor name="${prefix}_contactsensor_sensor" type="contact">
                         <always_on>true</always_on>
                         <update_rate>50</update_rate>
@@ -1565,5 +1565,5 @@
                                 ${prefix}_LOWER_LEG_fixed_joint_lump__${prefix}_FOOT_collision_1</collision>
                         </contact>
-                    </sensor>
+                    </sensor> -->
                 </gazebo>
             </xacro:if>
@@ -1740,5 +1740,5 @@
                         </surface>
                     </collision>
-                    <sensor name="${prefix}_contactsensor_sensor" type="contact">
+                    <!-- <sensor name="${prefix}_contactsensor_sensor" type="contact">
                         <always_on>true</always_on>
                         <update_rate>50</update_rate>
@@ -1747,5 +1747,5 @@
                                 ${prefix}_LOWER_LEG_fixed_joint_lump__${prefix}_FOOT_collision_1</collision>
                         </contact>
-                    </sensor>
+                    </sensor> -->
                 </gazebo>
             </xacro:if>
@@ -1922,5 +1922,5 @@
                         </surface>
                     </collision>
-                    <sensor name="${prefix}_contactsensor_sensor" type="contact">
+                    <!-- <sensor name="${prefix}_contactsensor_sensor" type="contact">
                         <always_on>true</always_on>
                         <update_rate>50</update_rate>
@@ -1929,5 +1929,5 @@
                                 ${prefix}_LOWER_LEG_fixed_joint_lump__${prefix}_FOOT_collision_1</collision>
                         </contact>
-                    </sensor>
+                    </sensor> -->
                 </gazebo>
             </xacro:if>
