Commit message: update omni mulinex urdf

File: urdf/links.xacro (robot description, xacro)
@@ -299,5 +299,5 @@
             <origin xyz="${hip_to_upper_leg_xyz}" rpy="${hip_to_upper_leg_rpy}" />
             <axis xyz="${axis}" />
-            <limit effort="5.0" lower="-${PI}" upper="${PI}" velocity="1000" />
+            <limit effort="5.0" lower="-${2*PI}" upper="${2*PI}" velocity="1000" />
             <!-- <dynamics damping="0.7" friction="100.0" /> -->
         </joint>
@@ -477,5 +477,5 @@
                 <origin xyz="${upper_to_lower_leg_xyz}" rpy="${upper_to_lower_leg_rpy}" />
                 <axis xyz="${axis}" />
-                <limit effort="5.0" lower="-${PI}" upper="${PI}" velocity="1000" />
+                <limit effort="5.0" lower="-${2*PI}" upper="${2*PI}" velocity="1000" />
                 <!-- <dynamics damping="0.7" friction="100.0" /> -->
             </joint>
@@ -739,5 +739,5 @@
                 <origin xyz="${upper_to_lower_leg_xyz}" rpy="${upper_to_lower_leg_rpy}" />
                 <axis xyz="${axis}" />
-                <limit effort="5.0" lower="-${PI}" upper="${PI}" velocity="1000" />
+                <limit effort="5.0" lower="-${2*PI}" upper="${2*PI}" velocity="1000" />
                 <!-- <dynamics damping="0.7" friction="100.0" /> -->
             </joint>
@@ -904,5 +904,5 @@
             </xacro:if>
             <!-- Omniwheels -->
-            <joint name="${prefix}_ANKLE" type="continuous">
+            <joint name="${prefix}_WHEEL_JNT" type="continuous">
                 <parent link="${prefix}_LOWER_LEG" />
                 <child link="${prefix}_WHEEL" />
@@ -3072,5 +3072,5 @@
                 <origin xyz="${upper_to_lower_leg_xyz}" rpy="${upper_to_lower_leg_rpy}" />
                 <axis xyz="${axis}" />
-                <limit effort="5.0" lower="-${PI}" upper="${PI}" velocity="1000" />
+                <limit effort="5.0" lower="-${2*PI}" upper="${2*PI}" velocity="1000" />
                 <!-- <dynamics damping="0.7" friction="100.0" /> -->
             </joint>
@@ -3507,5 +3507,5 @@
                 <origin xyz="${upper_to_lower_leg_xyz}" rpy="${upper_to_lower_leg_rpy}" />
                 <axis xyz="${axis}" />
-                <limit effort="5.0" lower="-${PI}" upper="${PI}" velocity="1000" />
+                <limit effort="5.0" lower="-${2*PI}" upper="${2*PI}" velocity="1000" />
                 <!-- <dynamics damping="0.7" friction="100.0" /> -->
             </joint>
@@ -3676,5 +3676,5 @@
             </xacro:if>
             <!-- Track wheels -->
-            <joint name="${prefix}_ANKLE" type="continuous">
+            <joint name="${prefix}_WHEEL_JNT" type="continuous">
                 <parent link="${prefix}_LOWER_LEG" />
                 <child link="${prefix}_WHEEL_1" />

File: urdf/mulinex.xacro (robot description, xacro)
@@ -78,13 +78,13 @@
         </gazebo>
         <gazebo>
-            <plugin filename="libgazebo_ros2_control.so" name="gazebo_ros2_control">
-                <parameters>$(find mulinex_gazebo)/config/mulinex_gazebo_sim_jnt_PD_IMU.yaml</parameters>
+            <plugin filename="gz_ros2_control-system" name="gz_ros2_control::GazeboSimROS2ControlPlugin">
+                <parameters>$(find mulinex_ignition)/config/mulinex_mf.yaml</parameters>
             </plugin>
         </gazebo>
         <ros2_control name="GazeboSystem" type="system">
             <hardware>
-                <plugin>gazebo_ros2_control/GazeboSystem</plugin>
+                <plugin>gz_ros2_control/GazeboSimSystem</plugin>
             </hardware>
-            <joint name="LH_HAA">
+            <!-- <joint name="LH_HAA">
                 <command_interface name="effort" />
                 <state_interface name="position">
@@ -95,26 +95,86 @@
                 </state_interface>
                 <state_interface name="effort" />
-            </joint>
+            </joint> -->
             <joint name="LH_HFE">
+                <command_interface name="position" />
+                <state_interface name="position">
+                    <param name="initial_value">$(arg LH_HFE)</param>
+                </state_interface>
+                <state_interface name="velocity">
+                    <param name="initial_value">0.0</param>
+                </state_interface>
+                <state_interface name="effort" />
+            </joint>
+            <joint name="LH_KFE">
+                <command_interface name="position" />
+                <state_interface name="position">
+                    <param name="initial_value">$(arg LH_KFE)</param>
+                </state_interface>
+                <state_interface name="velocity">
+                    <param name="initial_value">0.0</param>
+                </state_interface>
+                <state_interface name="effort" />
+            </joint>
+            <!-- <joint name="LF_HAA">
                 <command_interface name="effort" />
                 <state_interface name="position">
-                    <param name="initial_value">$(arg LH_HFE)</param>
-                </state_interface>
-                <state_interface name="velocity">
-                    <param name="initial_value">0.0</param>
-                </state_interface>
-                <state_interface name="effort" />
-            </joint>
-            <joint name="LH_KFE">
+                    <param name="initial_value">$(arg front_haa)</param>
+                </state_interface>
+                <state_interface name="velocity">
+                    <param name="initial_value">0.0</param>
+                </state_interface>
+                <state_interface name="effort" />
+            </joint> -->
+            <joint name="LF_HFE">
+                <command_interface name="position" />
+                <state_interface name="position">
+                    <param name="initial_value">$(arg LF_HFE)</param>
+                </state_interface>
+                <state_interface name="velocity">
+                    <param name="initial_value">0.0</param>
+                </state_interface>
+                <state_interface name="effort" />
+            </joint>
+            <joint name="LF_KFE">
+                <command_interface name="position" />
+                <state_interface name="position">
+                    <param name="initial_value">$(arg LF_KFE)</param>
+                </state_interface>
+                <state_interface name="velocity">
+                    <param name="initial_value">0.0</param>
+                </state_interface>
+                <state_interface name="effort" />
+            </joint>
+            <!-- <joint name="RH_HAA">
                 <command_interface name="effort" />
                 <state_interface name="position">
-                    <param name="initial_value">$(arg LH_KFE)</param>
-                </state_interface>
-                <state_interface name="velocity">
-                    <param name="initial_value">0.0</param>
-                </state_interface>
-                <state_interface name="effort" />
-            </joint>
-            <joint name="LF_HAA">
+                    <param name="initial_value">$(arg hind_haa)</param>
+                </state_interface>
+                <state_interface name="velocity">
+                    <param name="initial_value">0.0</param>
+                </state_interface>
+                <state_interface name="effort" />
+            </joint> -->
+            <joint name="RH_HFE">
+                <command_interface name="position" />
+                <state_interface name="position">
+                    <param name="initial_value">$(arg RH_HFE)</param>
+                </state_interface>
+                <state_interface name="velocity">
+                    <param name="initial_value">0.0</param>
+                </state_interface>
+                <state_interface name="effort" />
+            </joint>
+            <joint name="RH_KFE">
+                <command_interface name="position" />
+                <state_interface name="position">
+                    <param name="initial_value">$(arg RH_KFE)</param>
+                </state_interface>
+                <state_interface name="velocity">
+                    <param name="initial_value">0.0</param>
+                </state_interface>
+                <state_interface name="effort" />
+            </joint>
+            <!-- <joint name="RF_HAA">
                 <command_interface name="effort" />
                 <state_interface name="position">
@@ -125,67 +185,7 @@
                 </state_interface>
                 <state_interface name="effort" />
-            </joint>
-            <joint name="LF_HFE">
-                <command_interface name="effort" />
-                <state_interface name="position">
-                    <param name="initial_value">$(arg LF_HFE)</param>
-                </state_interface>
-                <state_interface name="velocity">
-                    <param name="initial_value">0.0</param>
-                </state_interface>
-                <state_interface name="effort" />
-            </joint>
-            <joint name="LF_KFE">
-                <command_interface name="effort" />
-                <state_interface name="position">
-                    <param name="initial_value">$(arg LF_KFE)</param>
-                </state_interface>
-                <state_interface name="velocity">
-                    <param name="initial_value">0.0</param>
-                </state_interface>
-                <state_interface name="effort" />
-            </joint>
-            <joint name="RH_HAA">
-                <command_interface name="effort" />
-                <state_interface name="position">
-                    <param name="initial_value">$(arg hind_haa)</param>
-                </state_interface>
-                <state_interface name="velocity">
-                    <param name="initial_value">0.0</param>
-                </state_interface>
-                <state_interface name="effort" />
-            </joint>
-            <joint name="RH_HFE">
-                <command_interface name="effort" />
-                <state_interface name="position">
-                    <param name="initial_value">$(arg RH_HFE)</param>
-                </state_interface>
-                <state_interface name="velocity">
-                    <param name="initial_value">0.0</param>
-                </state_interface>
-                <state_interface name="effort" />
-            </joint>
-            <joint name="RH_KFE">
-                <command_interface name="effort" />
-                <state_interface name="position">
-                    <param name="initial_value">$(arg RH_KFE)</param>
-                </state_interface>
-                <state_interface name="velocity">
-                    <param name="initial_value">0.0</param>
-                </state_interface>
-                <state_interface name="effort" />
-            </joint>
-            <joint name="RF_HAA">
-                <command_interface name="effort" />
-                <state_interface name="position">
-                    <param name="initial_value">$(arg front_haa)</param>
-                </state_interface>
-                <state_interface name="velocity">
-                    <param name="initial_value">0.0</param>
-                </state_interface>
-                <state_interface name="effort" />
-            </joint>
+            </joint> -->
             <joint name="RF_HFE">
-                <command_interface name="effort" />
+                <command_interface name="position" />
                 <state_interface name="position">
                     <param name="initial_value">$(arg RF_HFE)</param>
@@ -197,5 +197,5 @@
             </joint>
             <joint name="RF_KFE">
-                <command_interface name="effort" />
+                <command_interface name="position" />
                 <state_interface name="position">
                     <param name="initial_value">$(arg RF_KFE)</param>
@@ -206,6 +206,46 @@
                 <state_interface name="effort" />
             </joint>
+             <joint name="RF_WHEEL_JNT">
+                <command_interface name="velocity" />
+                <state_interface name="position">
+                    <param name="initial_value">0.0</param>
+                </state_interface>
+                <state_interface name="velocity">
+                    <param name="initial_value">0.0</param>
+                </state_interface>
+                <state_interface name="effort" />
+            </joint>
+             <joint name="RH_WHEEL_JNT">
+                <command_interface name="velocity" />
+                <state_interface name="position">
+                    <param name="initial_value">0.0</param>
+                </state_interface>
+                <state_interface name="velocity">
+                    <param name="initial_value">0.0</param>
+                </state_interface>
+                <state_interface name="effort" />
+            </joint>
+            <joint name="LF_WHEEL_JNT">
+                <command_interface name="velocity" />
+                <state_interface name="position">
+                    <param name="initial_value">0.0</param>
+                </state_interface>
+                <state_interface name="velocity">
+                    <param name="initial_value">0.0</param>
+                </state_interface>
+                <state_interface name="effort" />
+            </joint>
+            <joint name="LH_WHEEL_JNT">
+                <command_interface name="velocity" />
+                <state_interface name="position">
+                    <param name="initial_value">0.0</param>
+                </state_interface>
+                <state_interface name="velocity">
+                    <param name="initial_value">0.0</param>
+                </state_interface>
+                <state_interface name="effort" />
+            </joint>
         </ros2_control>
-        <gazebo reference="base_link">
+        <!-- <gazebo reference="base_link">
             <sensor name="br_imu" type="imu">
                 <always_on>true</always_on>
@@ -253,5 +293,5 @@
                 </linear_acceleration>
                 </imu>
-                <!-- <plugin name="bytes_imu" filename="libgazebo_ros_imu_sensor.so">
+                <plugin name="bytes_imu" filename="libgazebo_ros_imu_sensor.so">
                     <ros>
                         <namespace>imu</namespace>
@@ -259,7 +299,7 @@
                     </ros>
                     <initial_orientation_as_reference>false</initial_orientation_as_reference>
-                </plugin> -->
+                </plugin>
             </sensor>
-        </gazebo>
+        </gazebo> -->
     </xacro:if>
 </robot>

Commit message: update omnicar urdf, add lidar, rgbd camera

File: urdf/links.xacro (robot description, xacro)
@@ -19,6 +19,4 @@
     <xacro:property name="PI" value="3.141592" />
     <!-- MULINEX VISUALIZATION meshes -->
-    <xacro:property name="mulinex_base"
-        value="file://$(find mulinex_description)/meshes//Body.stl" />
     <xacro:property name="mulinex_module_left_front"
         value="file://$(find mulinex_description)/meshes//Module_left_front.stl" />

File: urdf/material.xacro (robot description, xacro)
@@ -14,5 +14,5 @@
   </material>
   <material name="orange">
-    <color rgba="${255/255} ${108/255} ${10/255} 0.5"/>
+    <color rgba="${255/255} ${108/255} ${10/255} 1.0"/>
   </material>
   <material name="brown">

File: urdf/omni_car_module.xacro (robot description, xacro)
@@ -1,5 +1,5 @@
 <?xml version="1.0"?>
 <robot xmlns:xacro="http://ros.org/wiki/xacro">
-    <xacro:include filename="$(find mulinex_description)/urdf/links.xacro" />
+    <xacro:include filename="$(find mulinex_description)/urdf/hip_module.xacro" />
     <xacro:include filename="$(find mulinex_description)/urdf/wheel.xacro" />
     <xacro:property name="PI" value="3.141592" />
@@ -17,5 +17,4 @@
             gazebo="${gazebo}"
         />
-        <!-- Lower leg link -->
     </xacro:macro>
 </robot>

File: urdf/omnicar.xacro (robot description, xacro)
@@ -2,28 +2,19 @@
 <robot name="mulinex" xmlns:xacro="http://ros.org/wiki/xacro">
     <xacro:include filename="$(find mulinex_description)/urdf/omni_car_module.xacro" />
-    <!-- <xacro:include filename="$(find mulinex_description)/urdf/material.xacro" /> -->
-    <xacro:include filename="$(find mulinex_description)/urdf/omnicar_gazebo.xacro" />
+    <xacro:property name="mulinex_base" value="file://$(find mulinex_description)/meshes//Body.stl" />
+    <xacro:include filename="$(find mulinex_description)/urdf/material.xacro" />
     <xacro:include filename="$(find mulinex_description)/urdf/omnicar_ignition.xacro" />
+    <xacro:include filename="$(find mulinex_description)/urdf/imu_sensor.xacro" />
+    <xacro:include filename="$(find mulinex_description)/urdf/lidar_sensor.xacro" />
+    <xacro:include filename="$(find mulinex_description)/urdf/camera_sensor.xacro" />
     <xacro:arg name="use_gazebo" default="true" />
-    <xacro:arg name="use_ignition" default="true" />
-    <xacro:arg name="simplify_meshes_lower_leg" default="true"/>
+    <xacro:arg name="yaml_file" default=""/>
+    <xacro:arg name="lidar_3D" default="true"/>
     <xacro:arg name="jnt_prefix" default=""/>
-    <!-- use "normal" if normal feet are used
-        use "omni" if omniwheels are used
-        use "goat" if goat feet are used
-        use "track" if track feet are used -->
     <xacro:arg name="front_haa" default="0.0" />
     <xacro:arg name="hind_haa" default="0.0" />
-    <xacro:arg name="RH_HFE" default="0.0" />
-    <xacro:arg name="RH_KFE" default="0.0" />
-    <xacro:arg name="RF_HFE" default="0.0" />
-    <xacro:arg name="RF_KFE" default="0.0" />
-    <xacro:arg name="LH_HFE" default="0.0" />
-    <xacro:arg name="LH_KFE" default="0.0" />
-    <xacro:arg name="LF_HFE" default="0.0" />
-    <xacro:arg name="LF_KFE" default="0.0" />
     <link name="$(arg jnt_prefix)base_link">
         <visual>
-            <material name="white" />
+            <material name="black"/>
             <origin xyz="0 0 0" rpy="0 0 0" />
             <geometry>
@@ -50,5 +41,5 @@
         gazebo="$(arg use_gazebo)"
         jnt_pref="$(arg jnt_prefix)"
-        simplify_meshes="$(arg simplify_meshes_lower_leg)"
+        simplify_meshes="true"
         />
     <xacro:omni_mod
@@ -56,5 +47,5 @@
         gazebo="$(arg use_gazebo)"
         jnt_pref="$(arg jnt_prefix)"
-        simplify_meshes="$(arg simplify_meshes_lower_leg)"
+        simplify_meshes="true"
         />
     <xacro:omni_mod
@@ -62,5 +53,5 @@
         gazebo="$(arg use_gazebo)"
         jnt_pref="$(arg jnt_prefix)"
-        simplify_meshes="$(arg simplify_meshes_lower_leg)"
+        simplify_meshes="true"
         />
     <xacro:omni_mod
@@ -68,14 +59,12 @@
         gazebo="$(arg use_gazebo)"
         jnt_pref="$(arg jnt_prefix)"
-        simplify_meshes="$(arg simplify_meshes_lower_leg)"
+        simplify_meshes="true"
     />
-    <xacro:if value="$(arg use_gazebo)">
-        <xacro:if value="$(arg use_ignition)">
-            <xacro:omnicar_ign_hw
-                gazebo="$(arg use_ignition)"
-            />
-        </xacro:if>
-        <xacro:unless value="$(arg use_ignition)">
-        </xacro:unless>
-    </xacro:if>
+    <xacro:imu_sensor/>
+    <xacro:lidar_sensor tredi="$(arg lidar_3D)"/>
+    <xacro:camera_sensor/>
+    <xacro:omnicar_ign_hw
+        gazebo="$(arg use_gazebo)"
+        yaml="$(arg yaml_file)"
+    />
 </robot>

File: urdf/omnicar_ignition.xacro (robot description, xacro)
@@ -1,9 +1,5 @@
 <?xml version="1.0"?>
 <robot xmlns:xacro="http://ros.org/wiki/xacro">
-    <xacro:include filename="$(find mulinex_description)/urdf/material.xacro" />
-    <xacro:macro name="omnicar_ign_hw" params="gazebo ">
-        <gazebo reference="base_link">
-            <material>Gazebo/White</material>
-        </gazebo>
+    <xacro:macro name="omnicar_ign_hw" params="gazebo yaml">
         <ros2_control name="GazeboSystem" type="system">
             <hardware>
