Commit message: update omnicar urdf, add lidar, rgbd camera

File: urdf/wheel.xacro (robot description, xacro)
@@ -4,1932 +4,1771 @@
     <!-- Transformation based on the position of each link -->
      <!-- WHEEL Hip -->
-        <xacro:property name="HAA_2_HFE_x" value="${190.0 * 0.001}" />
-        <xacro:property name="HAA_2_HFE_y" value="${25.0 * 0.001}" />
+    <xacro:property name="mulinex_roller"
+        value="file://$(find mulinex_description)/meshes//roller_1.STL" />
+    <xacro:property name="mulinex_mec_wheel_LF"
+        value="file://$(find mulinex_description)/meshes//mecanum_wheel_lf.STL" />
+    <xacro:property name="mulinex_mec_wheel_RF"
+        value="file://$(find mulinex_description)/meshes//mecanum_wheel_rf.STL" />
+    <xacro:property name="mulinex_mec_wheel_LH"
+        value="file://$(find mulinex_description)/meshes//mecanum_wheel_lh.STL" />
+    <xacro:property name="mulinex_mec_wheel_RH"
+        value="file://$(find mulinex_description)/meshes//mecanum_wheel_rh.STL" />
+    <xacro:property name="HAA_2_HFE_x" value="${190.0 * 0.001}" />
+    <xacro:property name="HAA_2_HFE_y" value="${25.0 * 0.001}" />
         <!-- Transformation based on the position of each link -->
     <xacro:macro name="wheel" params="prefix gazebo">
         <joint name="${prefix}_WHEEL_JNT" type="continuous">
-                <parent link="${prefix}_SHOULDER" />
-                <child link="${prefix}_WHEEL" />
+            <parent link="${prefix}_SHOULDER" />
+            <child link="${prefix}_WHEEL" />
+            <xacro:if value="${prefix == 'LF'}">
+                <origin xyz="${HAA_2_HFE_x} ${HAA_2_HFE_y} 0" rpy="0 0 0" />
+                <axis xyz="0 1 0" />
+            </xacro:if>
+            <xacro:if value="${prefix == 'LH'}">
+                <origin xyz="${-HAA_2_HFE_x} ${HAA_2_HFE_y} 0" rpy="0 0 0" />
+                <axis xyz="0 1 0" />
+            </xacro:if>
+            <xacro:if value="${prefix == 'RF'}">
+                <origin xyz="${HAA_2_HFE_x} ${-HAA_2_HFE_y} 0" rpy="0 0 0" />
+                <axis xyz="0 -1 0" />
+            </xacro:if>
+            <xacro:if value="${prefix == 'RH'}">
+                <origin xyz="${-HAA_2_HFE_x} ${-HAA_2_HFE_y} 0" rpy="0 0 0" />
+                <axis xyz="0 -1 0" />
+            </xacro:if>
+        </joint>
+        <link name="${prefix}_WHEEL">
+            <visual>
+                <material name="black" />
                 <xacro:if value="${prefix == 'LF'}">
-                    <origin xyz="${HAA_2_HFE_x} ${HAA_2_HFE_y} 0" rpy="0 0 0" />
-                    <axis xyz="0 1 0" />
+                    <origin xyz="0 0 0" rpy="0 0 0" />
+                    <geometry>
+                        <mesh filename="${mulinex_mec_wheel_LF}" />
+                    </geometry>
                 </xacro:if>
                 <xacro:if value="${prefix == 'LH'}">
-                    <origin xyz="${-HAA_2_HFE_x} ${HAA_2_HFE_y} 0" rpy="0 0 0" />
-                    <axis xyz="0 1 0" />
+                    <origin xyz="0 0  0" rpy="0 0 0" />
+                    <geometry>
+                        <mesh filename="${mulinex_mec_wheel_LH}" />
+                    </geometry>
                 </xacro:if>
                 <xacro:if value="${prefix == 'RF'}">
-                    <origin xyz="${HAA_2_HFE_x} ${-HAA_2_HFE_y} 0" rpy="0 0 0" />
-                    <axis xyz="0 -1 0" />
+                    <origin xyz="0 0 0" rpy="0 0 0" />
+                    <geometry>
+                        <mesh filename="${mulinex_mec_wheel_RF}" />
+                    </geometry>
                 </xacro:if>
                 <xacro:if value="${prefix == 'RH'}">
-                    <origin xyz="${-HAA_2_HFE_x} ${-HAA_2_HFE_y} 0" rpy="0 0 0" />
-                    <axis xyz="0 -1 0" />
-                </xacro:if>
-            </joint>
-        <link name="${prefix}_WHEEL">
-                <visual>
-                    <material name="white" />
-                    <xacro:if value="${prefix == 'LF'}">
-                        <origin xyz="0 0 0" rpy="0 0 0" />
-                        <geometry>
-                            <mesh filename="${mulinex_mec_wheel_LF}" />
-                        </geometry>
-                    </xacro:if>
-                    <xacro:if value="${prefix == 'LH'}">
-                        <origin xyz="0 0  0" rpy="0 0 0" />
-                        <geometry>
-                            <mesh filename="${mulinex_mec_wheel_LH}" />
-                        </geometry>
-                    </xacro:if>
-                    <xacro:if value="${prefix == 'RF'}">
-                        <origin xyz="0 0 0" rpy="0 0 0" />
-                        <geometry>
-                            <mesh filename="${mulinex_mec_wheel_RF}" />
-                        </geometry>
-                    </xacro:if>
-                    <xacro:if value="${prefix == 'RH'}">
-                        <origin xyz="0 0 0" rpy="0 0 0" />
-                        <geometry>
-                            <mesh filename="${mulinex_mec_wheel_RH}" />
-                        </geometry>
-                    </xacro:if>
-                </visual>
-                <!-- NO COLLISION FOR THE MECHANUM WHEELS -->
-                <inertial>
-                    <xacro:if value="${prefix == 'LF'}">
-                        <origin xyz="0 0.047255 -2.335E-07" rpy="0 0 0" />
-                        <mass value="0.078919" />
-                        <inertia ixx="4.9627E-05" ixy="1.7873E-11"
-                            ixz="-2.2576E-09" iyy="7.8948E-05"
-                            iyz="-7.6317E-12" izz="4.9622E-05" />
-                    </xacro:if>
-                    <xacro:if value="${prefix == 'LH'}">
-                        <origin xyz="0 0.047255 -1.5525E-07" rpy="0 0 0" />
-                        <mass value="0.078525" />
-                        <inertia ixx="4.9627E-05" ixy="-2.1009E-12"
-                            ixz="-1.8882E-09" iyy="7.8948E-05"
-                            iyz="4.4431E-12" izz="4.9622E-05" />
-                    </xacro:if>
-                    <xacro:if value="${prefix == 'RF'}">
-                        <origin xyz="0 -0.047255 -1.5525E-07" rpy="0 0 0" />
-                        <mass value="0.078525" />
-                        <inertia ixx="4.9627E-05" ixy="-2.1009E-12"
-                            ixz="1.8882E-09" iyy="7.8948E-05"
-                            iyz="-4.4431E-12" izz="4.9622E-05" />
-                    </xacro:if>
-                    <xacro:if value="${prefix == 'RH'}">
-                        <origin xyz="0 -0.047255 -2.3351E-07" rpy="0 0 0" />
-                        <mass value="0.078919" />
-                        <inertia ixx="4.9627E-05" ixy="1.7873E-11"
-                            ixz="-2.2576E-09" iyy="7.8948E-05"
-                            iyz="-7.6317E-12" izz="4.9622E-05" />
-                    </xacro:if>
-                </inertial>
-            </link>
-            <xacro:if value="${gazebo}">
-                <gazebo reference="${prefix}_WHEEL">
-                    <material>Gazebo/White</material>
-                    <collision>
-                        <surface>
-                            <friction>
-                                <ode>
-                                    <mu>0.6</mu>
-                                    <mu2>0.6</mu2>
-                                    <slip1>0</slip1>
-                                    <slip2>0</slip2>
-                                </ode>
-                            </friction>
-                            <contact>
-                                <ode>
-                                    <kp>10000.0</kp>
-                                    <kd>100.0</kd>
-                                    <min_depth>0.001</min_depth>
-                                </ode>
-                            </contact>
-                        </surface>
-                    </collision>
-                </gazebo>
-            </xacro:if>
-            <link name="${prefix}_Roller1">
+                    <origin xyz="0 0 0" rpy="0 0 0" />
+                    <geometry>
+                        <mesh filename="${mulinex_mec_wheel_RH}" />
+                    </geometry>
+                </xacro:if>
+            </visual>
+            <!-- NO COLLISION FOR THE MECHANUM WHEELS -->
+            <inertial>
                 <xacro:if value="${prefix == 'LF'}">
-                    <inertial>
-                        <origin
-                            xyz="0 0 6.3075E-15"
-                            rpy="0 0 0" />
-                        <mass
-                            value="0.0059616" />
-                        <inertia
-                            ixx="7.911E-07"
-                            ixy="1.2914E-12"
-                            ixz="1.2242E-22"
-                            iyy="7.9113E-07"
-                            iyz="-5.294E-23"
-                            izz="2.3532E-07" />
-                    </inertial>
-                    <visual>
-                        <origin
-                            xyz="0 0 0"
-                            rpy="0 0 0" />
-                        <geometry>
-                            <mesh filename="${mulinex_roller}" />
-                        </geometry>
-                        <material
-                            name="">
-                            <color
-                                rgba="0.29804 0.29804 0.29804 1" />
-                        </material>
-                    </visual>
-                    <collision>
-                        <origin
-                            xyz="0 0 0"
-                            rpy="0 0 0" />
-                        <geometry>
-                            <mesh filename="${mulinex_roller}" />
-                        </geometry>
-                    </collision>
+                    <origin xyz="0 0.047255 -2.335E-07" rpy="0 0 0" />
+                    <mass value="0.078919" />
+                    <inertia ixx="4.9627E-05" ixy="1.7873E-11"
+                        ixz="-2.2576E-09" iyy="7.8948E-05"
+                        iyz="-7.6317E-12" izz="4.9622E-05" />
+                </xacro:if>
+                <xacro:if value="${prefix == 'LH'}">
+                    <origin xyz="0 0.047255 -1.5525E-07" rpy="0 0 0" />
+                    <mass value="0.078525" />
+                    <inertia ixx="4.9627E-05" ixy="-2.1009E-12"
+                        ixz="-1.8882E-09" iyy="7.8948E-05"
+                        iyz="4.4431E-12" izz="4.9622E-05" />
                 </xacro:if>
                 <xacro:if value="${prefix == 'RF'}">
-                    <inertial>
-                        <origin
-                            xyz="0 0 0"
-                            rpy="0 0 0" />
-                        <mass
-                            value="0.0059616" />
-                        <inertia
-                            ixx="7.911E-07"
-                            ixy="1.2914E-12"
-                            ixz="2.5808E-22"
-                            iyy="7.9113E-07"
-                            iyz="-5.4263E-22"
-                            izz="2.3532E-07" />
-                    </inertial>
-                    <visual>
-                        <origin
-                            xyz="0 0 0"
-                            rpy="0 0 0" />
-                        <geometry>
-                            <mesh filename="${mulinex_roller}" />
-                        </geometry>
-                        <material
-                            name="">
-                            <color
-                                rgba="0.29804 0.29804 0.29804 1" />
-                        </material>
-                    </visual>
-                    <collision>
-                        <origin
-                            xyz="0 0 0"
-                            rpy="0 0 0" />
-                        <geometry>
-                            <mesh filename="${mulinex_roller}" />
-                        </geometry>
-                    </collision>
-                </xacro:if>
-                <xacro:if value="${prefix == 'LH'}">
-                    <inertial>
-                        <origin
-                            xyz="0 0 6.3075E-15"
-                            rpy="0 0 0" />
-                        <mass
-                            value="0.0059616" />
-                        <inertia
-                            ixx="7.911E-07"
-                            ixy="1.2914E-12"
-                            ixz="1.9521E-22"
-                            iyy="7.9113E-07"
-                            iyz="-5.0954E-22"
-                            izz="2.3532E-07" />
-                    </inertial>
-                    <visual>
-                        <origin
-                            xyz="0 0 0"
-                            rpy="0 0 0" />
-                        <geometry>
-                            <mesh filename="${mulinex_roller}" />
-                        </geometry>
-                        <material
-                            name="">
-                            <color
-                                rgba="0.29804 0.29804 0.29804 1" />
-                        </material>
-                    </visual>
-                    <collision>
-                        <origin
-                            xyz="0 0 0"
-                            rpy="0 0 0" />
-                        <geometry>
-                            <mesh filename="${mulinex_roller}" />
-                        </geometry>
-                    </collision>
+                    <origin xyz="0 -0.047255 -1.5525E-07" rpy="0 0 0" />
+                    <mass value="0.078525" />
+                    <inertia ixx="4.9627E-05" ixy="-2.1009E-12"
+                        ixz="1.8882E-09" iyy="7.8948E-05"
+                        iyz="-4.4431E-12" izz="4.9622E-05" />
                 </xacro:if>
                 <xacro:if value="${prefix == 'RH'}">
-                    <inertial>
-                        <origin
-                            xyz="0 0 6.3075E-15"
-                            rpy="0 0 0" />
-                        <mass
-                            value="0.0059616" />
-                        <inertia
-                            ixx="7.911E-07"
-                            ixy="1.2914E-12"
-                            ixz="1.2242E-22"
-                            iyy="7.9113E-07"
-                            iyz="-5.294E-23"
-                            izz="2.3532E-07" />
-                    </inertial>
-                    <visual>
-                        <origin
-                            xyz="0 0 0"
-                            rpy="0 0 0" />
-                        <geometry>
-                            <mesh filename="${mulinex_roller}" />
-                        </geometry>
-                        <material
-                            name="">
-                            <color
-                                rgba="0.29804 0.29804 0.29804 1" />
-                        </material>
-                    </visual>
-                    <collision>
-                        <origin
-                            xyz="0 0 0"
-                            rpy="0 0 0" />
-                        <geometry>
-                            <mesh filename="${mulinex_roller}" />
-                        </geometry>
-                    </collision>
-                </xacro:if>
-            </link>
-            <xacro:if value="${gazebo}">
-                <gazebo reference="${prefix}_Roller1">
-                    <material>Gazebo/White</material>
-                    <collision>
-                        <surface>
-                            <friction>
-                                <ode>
-                                    <mu>0.6</mu>
-                                    <mu2>0.6</mu2>
-                                    <slip1>0</slip1>
-                                    <slip2>0</slip2>
-                                </ode>
-                            </friction>
-                            <contact>
-                                <ode>
-                                    <kp>10000.0</kp>
-                                    <kd>100.0</kd>
-                                    <min_depth>0.001</min_depth>
-                                </ode>
-                            </contact>
-                        </surface>
-                    </collision>
-                    <!-- <sensor name="${prefix}_contactsensor_sensor" type="contact">
-                        <always_on>true</always_on>
-                        <update_rate>50</update_rate>
+                    <origin xyz="0 -0.047255 -2.3351E-07" rpy="0 0 0" />
+                    <mass value="0.078919" />
+                    <inertia ixx="4.9627E-05" ixy="1.7873E-11"
+                        ixz="-2.2576E-09" iyy="7.8948E-05"
+                        iyz="-7.6317E-12" izz="4.9622E-05" />
+                </xacro:if>
+            </inertial>
+        </link>
+        <xacro:if value="${gazebo}">
+            <gazebo reference="${prefix}_WHEEL">
+                <collision>
+                    <surface>
+                        <friction>
+                            <ode>
+                                <mu>0.6</mu>
+                                <mu2>0.6</mu2>
+                                <slip1>0</slip1>
+                                <slip2>0</slip2>
+                            </ode>
+                        </friction>
                         <contact>
-                            <collision>
-                                ${prefix}_LOWER_LEG_fixed_joint_lump__${prefix}_FOOT_collision_1</collision>
+                            <ode>
+                                <kp>1000.0</kp>
+                                <kd>10.0</kd>
+                                <min_depth>0.001</min_depth>
+                            </ode>
                         </contact>
-                    </sensor> -->
-                </gazebo>
-            </xacro:if>
-            <link name="${prefix}_Roller2">
-                <xacro:if value="${prefix == 'LF'}">
-                    <inertial>
-                        <origin
-                            xyz="0 0 6.3075E-15"
-                            rpy="0 0 0" />
-                        <mass
-                            value="0.0059616" />
-                        <inertia
-                            ixx="7.911E-07"
-                            ixy="1.2914E-12"
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
Commit message: Bug fix

File: urdf/links.xacro (robot description, xacro)
@@ -19,4 +19,6 @@
     <xacro:property name="PI" value="3.141592" />
     <!-- MULINEX VISUALIZATION meshes -->
+    <xacro:property name="mulinex_base"
+        value="file://$(find mulinex_description)/meshes//Body.stl" />
     <xacro:property name="mulinex_module_left_front"
         value="file://$(find mulinex_description)/meshes//Module_left_front.stl" />
