Commit message: Use effort interfaces in mulinex_white + use arg for controller yaml file + change axis of some mecanum wheel in mulinex

File: urdf/links.xacro (robot description, xacro)
@@ -923,9 +923,9 @@
                 <xacro:if value="${prefix == 'RF'}">
                     <origin xyz="${KFE_2_FOOT_x} -0.01145 0" rpy="0 0 0" />
-                    <axis xyz="0 1 0" />
+                    <axis xyz="0 -1 0" />
                 </xacro:if>
                 <xacro:if value="${prefix == 'RH'}">
                     <origin xyz="${-KFE_2_FOOT_x} -0.01145 0" rpy="0 0 0" />
-                    <axis xyz="0 1 0" />
+                    <axis xyz="0 -1 0" />
                 </xacro:if>
             </joint>

File: urdf/mulinex.xacro (robot description, xacro)
@@ -5,4 +5,5 @@
     <xacro:include filename="$(find mulinex_description)/urdf/material.xacro" />
     <xacro:arg name="use_gazebo" default="false" />
+    <xacro:arg name="yaml_file" default="" />
     <xacro:arg name="simplify_meshes_lower_leg" default="true"/>
     <!-- use "normal" if normal feet are used
@@ -79,5 +80,5 @@
         <gazebo>
             <plugin filename="gz_ros2_control-system" name="gz_ros2_control::GazeboSimROS2ControlPlugin">
-                <parameters>$(find mulinex_ignition)/config/mulinex_mf.yaml</parameters>
+                <parameters>$(arg yaml_file)</parameters>
             </plugin>
         </gazebo>
@@ -97,5 +98,5 @@
             </joint> -->
             <joint name="LH_HFE">
-                <command_interface name="position" />
+                <command_interface name="effort" />
                 <state_interface name="position">
                     <param name="initial_value">$(arg LH_HFE)</param>
@@ -107,5 +108,5 @@
             </joint>
             <joint name="LH_KFE">
-                <command_interface name="position" />
+                <command_interface name="effort" />
                 <state_interface name="position">
                     <param name="initial_value">$(arg LH_KFE)</param>
@@ -127,5 +128,5 @@
             </joint> -->
             <joint name="LF_HFE">
-                <command_interface name="position" />
+                <command_interface name="effort" />
                 <state_interface name="position">
                     <param name="initial_value">$(arg LF_HFE)</param>
@@ -137,5 +138,5 @@
             </joint>
             <joint name="LF_KFE">
-                <command_interface name="position" />
+                <command_interface name="effort" />
                 <state_interface name="position">
                     <param name="initial_value">$(arg LF_KFE)</param>
@@ -157,5 +158,5 @@
             </joint> -->
             <joint name="RH_HFE">
-                <command_interface name="position" />
+                <command_interface name="effort" />
                 <state_interface name="position">
                     <param name="initial_value">$(arg RH_HFE)</param>
@@ -167,5 +168,5 @@
             </joint>
             <joint name="RH_KFE">
-                <command_interface name="position" />
+                <command_interface name="effort" />
                 <state_interface name="position">
                     <param name="initial_value">$(arg RH_KFE)</param>
@@ -187,5 +188,5 @@
             </joint> -->
             <joint name="RF_HFE">
-                <command_interface name="position" />
+                <command_interface name="effort" />
                 <state_interface name="position">
                     <param name="initial_value">$(arg RF_HFE)</param>
@@ -197,5 +198,5 @@
             </joint>
             <joint name="RF_KFE">
-                <command_interface name="position" />
+                <command_interface name="effort" />
                 <state_interface name="position">
                     <param name="initial_value">$(arg RF_KFE)</param>

File: urdf/mulinex_white.xacro (robot description, xacro)
@@ -5,4 +5,5 @@
     <xacro:include filename="$(find mulinex_description)/urdf/material.xacro" />
     <xacro:arg name="use_gazebo" default="false" />
+    <xacro:arg name="yaml_file" default="" />
     <xacro:arg name="simplify_meshes_lower_leg" default="true"/>
     <!-- use "normal" if normal feet are used
@@ -88,5 +89,5 @@
         <gazebo>
             <plugin filename="gz_ros2_control-system" name="gz_ros2_control::GazeboSimROS2ControlPlugin">
-                <parameters>$(find mulinex_ignition)/config/mulinex_mf.yaml</parameters>
+                <parameters>$(arg yaml_file)</parameters>
             </plugin>
         </gazebo>
@@ -96,5 +97,5 @@
             </hardware>
             <joint name="LH_HFE">
-                <command_interface name="position" />
+                <command_interface name="effort" />
                 <state_interface name="position">
                     <param name="initial_value">$(arg LH_HFE)</param>
@@ -106,5 +107,5 @@
             </joint>
             <joint name="LH_KFE">
-                <command_interface name="position" />
+                <command_interface name="effort" />
                 <state_interface name="position">
                     <param name="initial_value">$(arg LH_KFE)</param>
@@ -116,5 +117,5 @@
             </joint>
             <joint name="LF_HFE">
-                <command_interface name="position" />
+                <command_interface name="effort" />
                 <state_interface name="position">
                     <param name="initial_value">$(arg LF_HFE)</param>
@@ -126,5 +127,5 @@
             </joint>
             <joint name="LF_KFE">
-                <command_interface name="position" />
+                <command_interface name="effort" />
                 <state_interface name="position">
                     <param name="initial_value">$(arg LF_KFE)</param>
@@ -136,5 +137,5 @@
             </joint>
             <joint name="RH_HFE">
-                <command_interface name="position" />
+                <command_interface name="effort" />
                 <state_interface name="position">
                     <param name="initial_value">$(arg RH_HFE)</param>
@@ -146,5 +147,5 @@
             </joint>
             <joint name="RH_KFE">
-                <command_interface name="position" />
+                <command_interface name="effort" />
                 <state_interface name="position">
                     <param name="initial_value">$(arg RH_KFE)</param>
@@ -156,5 +157,5 @@
             </joint>
             <joint name="RF_HFE">
-                <command_interface name="position" />
+                <command_interface name="effort" />
                 <state_interface name="position">
                     <param name="initial_value">$(arg RF_HFE)</param>
@@ -166,5 +167,5 @@
             </joint>
             <joint name="RF_KFE">
-                <command_interface name="position" />
+                <command_interface name="effort" />
                 <state_interface name="position">
                     <param name="initial_value">$(arg RF_KFE)</param>

File: urdf/omnicar_gazebo.xacro (robot description, xacro)
@@ -8,5 +8,5 @@
         <gazebo>
             <plugin filename="libgazebo_ros2_control.so" name="gazebo_ros2_control">
-                <parameters>$(find mulinex_gazebo)/config/mulinex_gazebo_sim_jnt_PD_IMU.yaml</parameters>
+                <parameters>$(find omni_gazebo)/config/mulinex_gazebo_sim_jnt_PD_IMU.yaml</parameters>
             </plugin>
         </gazebo>

File: urdf/omnicar_ignition.xacro (robot description, xacro)
@@ -2,54 +2,56 @@
 <robot xmlns:xacro="http://ros.org/wiki/xacro">
     <xacro:macro name="omnicar_ign_hw" params="gazebo yaml">
-        <ros2_control name="GazeboSystem" type="system">
-            <hardware>
-                <plugin>gz_ros2_control/GazeboSimSystem</plugin>
-            </hardware>
-            <joint name="LH_WHEEL_JNT">
-                <command_interface name="velocity" />
-                <state_interface name="position">
-                    <param name="initial_value">0.0</param>
-                </state_interface>
-                <state_interface name="velocity">
-                    <param name="initial_value">0.0</param>
-                </state_interface>
-                <state_interface name="effort" />
-            </joint>
-            <joint name="LF_WHEEL_JNT">
-                <command_interface name="velocity" />
-                <state_interface name="position">
-                    <param name="initial_value"> 0.0</param>
-                </state_interface>
-                <state_interface name="velocity">
-                    <param name="initial_value">0.0</param>
-                </state_interface>
-                <state_interface name="effort" />
-            </joint>
-            <joint name="RH_WHEEL_JNT">
-                <command_interface name="velocity" />
-                <state_interface name="position">
-                    <param name="initial_value">0.0</param>
-                </state_interface>
-                <state_interface name="velocity">
-                    <param name="initial_value">0.0</param>
-                </state_interface>
-                <state_interface name="effort" />
-            </joint>
-            <joint name="RF_WHEEL_JNT">
-                <command_interface name="velocity" />
-                <state_interface name="position">
-                    <param name="initial_value">0.0</param>
-                </state_interface>
-                <state_interface name="velocity">
-                    <param name="initial_value">0.0</param>
-                </state_interface>
-                <state_interface name="effort" />
-            </joint>
-        </ros2_control>
-        <gazebo>
-            <plugin filename="gz_ros2_control-system" name="gz_ros2_control::GazeboSimROS2ControlPlugin">
-                <parameters>$(find mulinex_ignition)/config/omnicar.yaml</parameters>
-            </plugin>
-        </gazebo>
+        <xacro:if value="${gazebo}">
+            <ros2_control name="GazeboSystem" type="system">
+                <hardware>
+                    <plugin>gz_ros2_control/GazeboSimSystem</plugin>
+                </hardware>
+                <joint name="LH_WHEEL_JNT">
+                    <command_interface name="velocity" />
+                    <state_interface name="position">
+                        <param name="initial_value">0.0</param>
+                    </state_interface>
+                    <state_interface name="velocity">
+                        <param name="initial_value">0.0</param>
+                    </state_interface>
+                    <state_interface name="effort" />
+                </joint>
+                <joint name="LF_WHEEL_JNT">
+                    <command_interface name="velocity" />
+                    <state_interface name="position">
+                        <param name="initial_value">0.0</param>
+                    </state_interface>
+                    <state_interface name="velocity">
+                        <param name="initial_value">0.0</param>
+                    </state_interface>
+                    <state_interface name="effort" />
+                </joint>
+                <joint name="RH_WHEEL_JNT">
+                    <command_interface name="velocity" />
+                    <state_interface name="position">
+                        <param name="initial_value">0.0</param>
+                    </state_interface>
+                    <state_interface name="velocity">
+                        <param name="initial_value">0.0</param>
+                    </state_interface>
+                    <state_interface name="effort" />
+                </joint>
+                <joint name="RF_WHEEL_JNT">
+                    <command_interface name="velocity" />
+                    <state_interface name="position">
+                        <param name="initial_value">0.0</param>
+                    </state_interface>
+                    <state_interface name="velocity">
+                        <param name="initial_value">0.0</param>
+                    </state_interface>
+                    <state_interface name="effort" />
+                </joint>
+            </ros2_control>
+            <gazebo>
+                <plugin filename="gz_ros2_control-system" name="gz_ros2_control::GazeboSimROS2ControlPlugin">
+                    <parameters>${yaml}</parameters>
+                </plugin>
+            </gazebo>
+        </xacro:if>
     </xacro:macro>
 </robot>
